Commit message: added m2 urdf

File: legged_examples/legged_unitree/legged_unitree_description/urdf/common/materials.xacro (robot description, xacro)
@@ -28,3 +28,15 @@
         <color rgba="1.0 1.0 1.0 1.0"/>
     </material>
+    <material name="svan_black">
+        <color rgba="0.0 0.0 0.0 1.0"/>
+    </material>
+    <material name="svan_blue">
+        <color rgba="0.0 0.0 0.8 1.0"/>
+    </material>
+    <material name="svan_green">
+        <color rgba="0.024 0.251 0.169 1.0"/>
+    </material>
+    <material name="svan_grey">
+        <color rgba="0.5 0.5 0.5 1.0"/>
+    </material>
 </robot>

File: legged_examples/legged_unitree/legged_unitree_description/urdf/robot.xacro (robot description, xacro)
@@ -4,14 +4,20 @@
     <xacro:include filename="$(find legged_unitree_description)/urdf/common/materials.xacro"/>
     <xacro:include filename="$(find legged_unitree_description)/urdf/common/leg.xacro"/>
-    <xacro:include filename="$(find legged_unitree_description)/urdf/common/gazebo.xacro"/>
+    <xacro:include filename="$(find legged_unitree_description)/urdf/common/leg_m2.xacro"/>
+    <!-- <xacro:include filename="$(find legged_unitree_description)/urdf/common/gazebo.xacro"/> -->
     <xacro:include filename="$(find legged_unitree_description)/urdf/common/imu.xacro"/>
     <xacro:include filename="$(find legged_unitree_description)/urdf/$(arg robot_type)/const.xacro"/>
 <!--    <xacro:property name="mesh_path" value="../meshes"/>-->
-    <xacro:property name="mesh_path" value="$(find legged_unitree_description)/meshes/$(arg robot_type)"/>
+    <xacro:property name="mesh_path" value="file://$(find legged_unitree_description)/meshes/$(arg robot_type)"/>
     <link name="base">
         <visual>
             <origin rpy="0 0 0" xyz="0 0 0"/>
             <geometry>
-                <mesh filename="${mesh_path}/trunk.dae" scale="1 1 1"/>
+                <xacro:if value="${'$(arg robot_type)' == 'm2'}">
+                    <mesh filename="${mesh_path}/torso.STL" scale="1 1 1"/>
+                </xacro:if>
+                <xacro:if value="${'$(arg robot_type)' != 'm2'}">
+                    <mesh filename="${mesh_path}/trunk.dae" scale="1 1 1"/>
+                </xacro:if>
             </geometry>
         </visual>
@@ -19,5 +25,10 @@
             <origin rpy="0 0 0" xyz="0 0 0"/>
             <geometry>
-                <box size="${trunk_length} ${trunk_width} ${trunk_height}"/>
+                <xacro:if value="${'$(arg robot_type)' == 'm2'}">
+                    <mesh filename="${mesh_path}/torso.STL" scale="1 1 1"/>
+                </xacro:if>
+                <xacro:if value="${'$(arg robot_type)' != 'm2'}">
+                    <box size="${trunk_length} ${trunk_width} ${trunk_height}"/>
+                </xacro:if>
             </geometry>
         </collision>
@@ -32,15 +43,26 @@
     </link>
     <xacro:IMU connected_to="base" imu_name="base_imu" xyz="0. 0. 0." rpy="0. 0. 0."/>
-    <xacro:leg prefix="LF" mesh_path="${mesh_path}" mirror="1" mirror_dae="True" front_hind="1" front_hind_dae="True">
-        <origin rpy="0 0 0" xyz="${leg_offset_x} ${leg_offset_y} 0"/>
-    </xacro:leg>
-    <xacro:leg prefix="LH" mesh_path="${mesh_path}" mirror="1" mirror_dae="True" front_hind="-1" front_hind_dae="False">
-        <origin rpy="0 0 0" xyz="${-leg_offset_x} ${leg_offset_y} 0"/>
-    </xacro:leg>
-    <xacro:leg prefix="RF" mesh_path="${mesh_path}" mirror="-1" mirror_dae="False" front_hind="1" front_hind_dae="True">
-        <origin rpy="0 0 0" xyz="${leg_offset_x} ${-leg_offset_y} 0"/>
-    </xacro:leg>
-    <xacro:leg prefix="RH" mesh_path="${mesh_path}" mirror="-1" mirror_dae="False" front_hind="-1" front_hind_dae="False">
-        <origin rpy="0 0 0" xyz="${-leg_offset_x} ${-leg_offset_y} 0"/>
-    </xacro:leg>
+    <!-- leg xacro for m2  -->
+    <xacro:if value="${'$(arg robot_type)' == 'm2'}">
+        <xacro:leg_m2 name="FR" mirror="1" front_hind="1"  />
+        <xacro:leg_m2 name="RR" mirror="1" front_hind="-1" />
+        <xacro:leg_m2 name="RL" mirror="-1"  front_hind="-1" />
+        <xacro:leg_m2 name="FL" mirror="-1"  front_hind="1"  />
+    </xacro:if>
+    <!-- leg xacro for other robots -->
+    <xacro:if value="${'$(arg robot_type)' != 'm2'}">
+        <xacro:leg prefix="LF" mesh_path="${mesh_path}" mirror="1" mirror_dae="True" front_hind="1" front_hind_dae="True">
+            <origin rpy="0 0 0" xyz="${leg_offset_x} ${leg_offset_y} 0"/>
+        </xacro:leg>
+        <xacro:leg prefix="LH" mesh_path="${mesh_path}" mirror="1" mirror_dae="True" front_hind="-1" front_hind_dae="False">
+            <origin rpy="0 0 0" xyz="${-leg_offset_x} ${leg_offset_y} 0"/>
+        </xacro:leg>
+        <xacro:leg prefix="RF" mesh_path="${mesh_path}" mirror="-1" mirror_dae="False" front_hind="1" front_hind_dae="True">
+            <origin rpy="0 0 0" xyz="${leg_offset_x} ${-leg_offset_y} 0"/>
+        </xacro:leg>
+        <xacro:leg prefix="RH" mesh_path="${mesh_path}" mirror="-1" mirror_dae="False" front_hind="-1" front_hind_dae="False">
+            <origin rpy="0 0 0" xyz="${-leg_offset_x} ${-leg_offset_y} 0"/>
+        </xacro:leg>
+    </xacro:if>
+    <xacro:include filename="$(find legged_unitree_description)/urdf/common/gazebo_m2.xacro"/>
 </robot>
