Commit message: fixed joint names

File: legged_examples/legged_unitree/legged_unitree_description/urdf/common/gazebo_m2.xacro (robot description, xacro)
@@ -58,5 +58,5 @@
   </gazebo>
   <!-- FR foot -->
-  <gazebo reference="foot_FR">
+  <gazebo reference="RF_FOOT">
         <material>Gazebo/Black</material>
       <collision>
@@ -93,40 +93,40 @@
     </gazebo>
     <!-- FL foot -->
-    <gazebo reference="foot_FL">
-        <material>Gazebo/Black</material>
-      <collision>
-        <surface>
-          <bounce>
-            <restitution_coefficient>0</restitution_coefficient>
-            <threshold>1e+06</threshold>
-          </bounce>
-          <friction>
-            <torsional>
-              <coefficient>0.3</coefficient>
-            </torsional>
-            <ode>
-              <mu>100.0</mu>
-              <mu2>50</mu2>
-            </ode>
-            <bullet>
-              <rolling_friction>0.3</rolling_friction>
-              <friction2>50</friction2>
-            </bullet>
-          </friction>
-          <contact>
-            <bullet>
-              <kp>30000.0</kp>
-              <kd>1000.0</kd>
-            </bullet>
-            <ode>
-              <kp>30000.0</kp>
-              <kd>1000.0</kd>
-            </ode>
-          </contact>
-        </surface>
-      </collision>
-    </gazebo>
-    <!-- FL foot -->
-    <gazebo reference="foot_RL">
+    <gazebo reference="LF_FOOT">
+        <material>Gazebo/Black</material>
+      <collision>
+        <surface>
+          <bounce>
+            <restitution_coefficient>0</restitution_coefficient>
+            <threshold>1e+06</threshold>
+          </bounce>
+          <friction>
+            <torsional>
+              <coefficient>0.3</coefficient>
+            </torsional>
+            <ode>
+              <mu>100.0</mu>
+              <mu2>50</mu2>
+            </ode>
+            <bullet>
+              <rolling_friction>0.3</rolling_friction>
+              <friction2>50</friction2>
+            </bullet>
+          </friction>
+          <contact>
+            <bullet>
+              <kp>30000.0</kp>
+              <kd>1000.0</kd>
+            </bullet>
+            <ode>
+              <kp>30000.0</kp>
+              <kd>1000.0</kd>
+            </ode>
+          </contact>
+        </surface>
+      </collision>
+    </gazebo>
+    <!-- RL foot -->
+    <gazebo reference="LH_FOOT">
         <material>Gazebo/Black</material>
       <collision>
@@ -163,5 +163,5 @@
     </gazebo>
     <!-- RR foot -->
-    <gazebo reference="foot_RR">
+    <gazebo reference="RH_FOOT">
         <material>Gazebo/Black</material>
       <collision>
@@ -201,11 +201,11 @@
           <plugin name="contact_plugin" filename="libcontact_plugin_new.so">
             <link1>foot_FR</link1>
-            <link2>foot_FL</link2>
-            <link3>foot_RL</link3>
-            <link4>foot_RR</link4>
+            <link2>FL_FOOT</link2>
+            <link3>RL_FOOT</link3>
+            <link4>RR_FOOT</link4>
             <contact_model>0</contact_model>
           </plugin>
       </gazebo> -->
-      <gazebo reference="foot_FR">
+      <gazebo reference="RF_FOOT">
         <sensor name="FR_contact_sensor" type="contact">
           <always_on>1</always_on>
@@ -218,5 +218,5 @@
         </sensor>
       </gazebo>
-      <gazebo reference="foot_FL">
+      <gazebo reference="LF_FOOT">
         <sensor name="FL_contact_sensor" type="contact">
           <always_on>1</always_on>
@@ -225,9 +225,9 @@
           </plugin>
           <contact>
-            <collision>foot_FL_collision</collision>
-          </contact>
-        </sensor>
-      </gazebo>
-      <gazebo reference="foot_RL">
+            <collision>FL_FOOT_collision</collision>
+          </contact>
+        </sensor>
+      </gazebo>
+      <gazebo reference="LH_FOOT">
         <sensor name="RL_contact_sensor" type="contact">
           <always_on>1</always_on>
@@ -236,9 +236,9 @@
           </plugin>
           <contact>
-            <collision>foot_RL_collision</collision>
-          </contact>
-        </sensor>
-      </gazebo>
-      <gazebo reference="foot_RR">
+            <collision>RL_FOOT_collision</collision>
+          </contact>
+        </sensor>
+      </gazebo>
+      <gazebo reference="RH_FOOT">
         <sensor name="RR_contact_sensor" type="contact">
           <always_on>1</always_on>
@@ -247,5 +247,5 @@
           </plugin>
           <contact>
-            <collision>foot_RR_collision</collision>
+            <collision>RR_FOOT_collision</collision>
           </contact>
         </sensor>

File: legged_examples/legged_unitree/legged_unitree_description/urdf/common/leg_m2.xacro (robot description, xacro)
@@ -5,6 +5,19 @@
     <xacro:macro name="leg_m2" params="name mirror front_hind">
     <xacro:property name="STL_path" value="file://$(find legged_unitree_description)/meshes/m2"/>
-        <!-- hip_link-->
-        <link name="${name}_hip_link">
+        <!-- HAA_joint -->
+        <joint name="${name}_HAA" type="revolute">
+            <origin xyz="${front_hind*abd_j_com_x} ${mirror*abd_j_com_y} ${abd_j_com_z}" rpy="0 0 0" />
+            <parent link="base"/>
+            <child link="${name}_hip"/>
+            <xacro:if value="${(front_hind == 1)}">
+                <axis xyz="1 0 0"/>
+            </xacro:if>
+            <xacro:if value="${(front_hind == -1)}">
+                <axis xyz="-1 0 0"/>
+            </xacro:if>
+            <limit lower="${abd_j_lower}" upper="${abd_j_upper}" effort="${abd_j_effort}" velocity="${abd_j_velocity}"/>
+        </joint>
+        <!-- hip-->
+        <link name="${name}_hip">
             <inertial>
                 <origin xyz="${front_hind*abd_l_com_x} ${mirror*abd_l_com_y} ${abd_l_com_z}"  rpy="0 0 0" />
@@ -49,19 +62,19 @@
             </collision>
         </link>
-        <!-- HAA_joint -->
-        <joint name="${name}_HAA_joint" type="revolute">
-            <origin xyz="${front_hind*abd_j_com_x} ${mirror*abd_j_com_y} ${abd_j_com_z}" rpy="0 0 0" />
-            <parent link="base"/>
-            <child link="${name}_hip_link"/>
-            <xacro:if value="${(front_hind == 1)}">
-                <axis xyz="1 0 0"/>
+        <!-- HFE -->
+        <joint name="${name}_HFE" type="revolute">
+            <origin xyz="${front_hind*hip_j_com_x} ${mirror*hip_j_com_y} ${hip_j_com_z}" rpy="0 0 0" />
+            <parent link="${name}_hip"/>
+            <child link="${name}_thigh"/>
+            <xacro:if value="${(mirror == 1)}">
+                <axis xyz="0 1 0"/>
             </xacro:if>
-            <xacro:if value="${(front_hind == -1)}">
-                <axis xyz="-1 0 0"/>
+            <xacro:if value="${(mirror == -1)}">
+                <axis xyz="0 1 0"/>
             </xacro:if>
-            <limit lower="${abd_j_lower}" upper="${abd_j_upper}" effort="${abd_j_effort}" velocity="${abd_j_velocity}"/>
+            <limit lower="${hip_j_lower}" upper="${hip_j_upper}" effort="${hip_j_effort}" velocity="${hip_j_velocity}"/>
         </joint>
         <!-- thigh link -->
-        <link name="${name}_thigh_link">
+        <link name="${name}_thigh">
             <inertial>
                 <origin xyz="${front_hind*hip_l_com_x} ${-mirror*hip_l_com_y} ${hip_l_com_z}"  rpy="0 0 0" />
@@ -96,9 +109,9 @@
             </collision>
         </link>
-        <!-- HFE_joint -->
-        <joint name="${name}_HFE_joint" type="revolute">
-            <origin xyz="${front_hind*hip_j_com_x} ${mirror*hip_j_com_y} ${hip_j_com_z}" rpy="0 0 0" />
-            <parent link="${name}_hip_link"/>
-            <child link="${name}_thigh_link"/>
+        <!-- KFE -->
+        <joint name="${name}_KFE" type="revolute">
+            <origin xyz="${front_hind*knee_j_com_x} ${mirror*knee_j_com_y} ${knee_j_com_z}" rpy="0 0 0" />
+            <parent link="${name}_thigh"/>
+            <child link="${name}_calf"/>
             <xacro:if value="${(mirror == 1)}">
                 <axis xyz="0 1 0"/>
@@ -107,8 +120,8 @@
                 <axis xyz="0 1 0"/>
             </xacro:if>
-            <limit lower="${hip_j_lower}" upper="${hip_j_upper}" effort="${hip_j_effort}" velocity="${hip_j_velocity}"/>
+            <limit lower="${knee_j_lower}" upper="${knee_j_upper}" effort="${knee_j_effort}" velocity="${knee_j_velocity}"/>
         </joint>
-        <!-- shank_link-->
-        <link name="${name}_shank_link">
+        <!-- calf-->
+        <link name="${name}_calf">
             <inertial>
                 <origin xyz="${front_hind*knee_l_com_x} ${mirror*knee_l_com_y} ${knee_l_com_z}"  rpy="0 0 0" />
@@ -143,19 +156,15 @@
             </collision>
         </link>
-        <!-- KFE_joint -->
-        <joint name="${name}_KFE_joint" type="revolute">
-            <origin xyz="${front_hind*knee_j_com_x} ${mirror*knee_j_com_y} ${knee_j_com_z}" rpy="0 0 0" />
-            <parent link="${name}_thigh_link"/>
-            <child link="${name}_shank_link"/>
-            <xacro:if value="${(mirror == 1)}">
-                <axis xyz="0 1 0"/>
-            </xacro:if>
-            <xacro:if value="${(mirror == -1)}">
-                <axis xyz="0 1 0"/>
-            </xacro:if>
-            <limit lower="${knee_j_lower}" upper="${knee_j_upper}" effort="${knee_j_effort}" velocity="${knee_j_velocity}"/>
+        <!-- foot_fixed -->
+        <joint name="${name}_foot_fixed" type="fixed" dont_collapse="true">
+            <!-- <origin xyz="${foot_fixed_com_x} ${mirror*foot_fixed_com_y} ${foot_fixed_com_z}" rpy="0 0 0" /> -->
+            <origin xyz="${foot_fixed_com_x} ${mirror*foot_fixed_com_y} ${foot_fixed_com_z}"/>
+            <parent link="${name}_calf"/>
+            <child link="${name}_FOOT"/>
+            <!-- <axis xyz="0 0 1"/> -->
+            <!-- <limit lower="0" upper="0" effort="1000" velocity="0" />            -->
         </joint>
         <!-- foot-->
-        <link name="foot_${name}">
+        <link name="${name}_FOOT">
             <contact>
                 <friction_anchor/>
@@ -184,12 +193,7 @@
             </collision>
         </link>
-        <!-- foot_j -->
-        <joint name="${name}_foot_j" type="revolute">
-            <origin xyz="${foot_j_com_x} ${mirror*foot_j_com_y} ${foot_j_com_z}" rpy="0 0 0" />
-            <parent link="${name}_shank_link"/>
-            <child link="foot_${name}"/>
-            <axis xyz="0 0 1"/>
-            <limit lower="0" upper="0" effort="1000" velocity="0" />
-        </joint>
+        <gazebo reference="${name}_foot_fixed">
+            <disableFixedJointLumping>true</disableFixedJointLumping>
+        </gazebo>
      </xacro:macro>
 </robot>

File: legged_examples/legged_unitree/legged_unitree_description/urdf/m2/const.xacro (robot description, xacro)
@@ -113,8 +113,8 @@
 <xacro:property name="knee_j_upper" value="4.916297857"/>
 <xacro:property name="knee_j_velocity" value ="28.6"/>
-<!-- foot_j -->
-<xacro:property name="foot_j_com_x" value="-0.00351"/>
-<xacro:property name="foot_j_com_y" value="0"/>
-<xacro:property name="foot_j_com_z" value="-0.1901"/>
-<xacro:property name="foot_j_axis" value="0 0 1"/>
+<!-- foot_fixed -->
+<xacro:property name="foot_fixed_com_x" value="-0.00351"/>
+<xacro:property name="foot_fixed_com_y" value="0"/>
+<xacro:property name="foot_fixed_com_z" value="-0.1901"/>
+<xacro:property name="foot_fixed_axis" value="0 0 1"/>
 </robot>

File: legged_examples/legged_unitree/legged_unitree_description/urdf/robot.xacro (robot description, xacro)
@@ -45,8 +45,8 @@
     <!-- leg xacro for m2  -->
     <xacro:if value="${'$(arg robot_type)' == 'm2'}">
-        <xacro:leg_m2 name="FR" mirror="1" front_hind="1"  />
-        <xacro:leg_m2 name="RR" mirror="1" front_hind="-1" />
-        <xacro:leg_m2 name="RL" mirror="-1"  front_hind="-1" />
-        <xacro:leg_m2 name="FL" mirror="-1"  front_hind="1"  />
+        <xacro:leg_m2 name="RF" mirror="1" front_hind="1"  />
+        <xacro:leg_m2 name="RH" mirror="1" front_hind="-1" />
+        <xacro:leg_m2 name="LH" mirror="-1"  front_hind="-1" />
+        <xacro:leg_m2 name="LF" mirror="-1"  front_hind="1"  />
     </xacro:if>
     <!-- leg xacro for other robots -->

Commit message: fixed controller

File: legged_examples/legged_unitree/legged_unitree_description/urdf/common/gazebo_m2.xacro (robot description, xacro)
@@ -2,50 +2,50 @@
   <robot xmlns:xacro="http://www.ros.org/wiki/xacro">
     <gazebo>
-          <plugin name="motor_controller" filename="libmotor_controller.so">
-            <!--
-            <kp0>75</kp0>
-            <kp1>30.2</kp1>
-            <kp2>18.415</kp2> -->
-            <kp0>200.2</kp0>
-            <kp1>60.2</kp1>
-            <kp2>42.415</kp2>
-            <kd0>1</kd0>
-            <kd1>1.5</kd1>
-            <kd2>0.5</kd2>
-            <!--
-            <kp0>80</kp0>
-            <kp1>40</kp1>
-            <kp2>20</kp2>
-            <kd0>1</kd0>
-            <kd1>1</kd1>
-            <kd2>0.5</kd2> -->
-            <!--
-            <kp0>200</kp0>
-            <kp1>120</kp1>
-            <kp2>60</kp2>
-            <kd0>1</kd0>
-            <kd1>1</kd1>
-            <kd2>0.5</kd2> -->
-            <!-- adding higher gains for the swing leg -->
-            <kpsw0>300</kpsw0>
-            <kpsw1>300</kpsw1>
-            <kpsw2>300</kpsw2>
-            <kdsw0>6</kdsw0>
-            <kdsw1>6</kdsw1>
-            <kdsw2>6</kdsw2>
-          </plugin>
+      <plugin name="motor_controller" filename="libmotor_controller.so">
+        <!--
+        <kp0>75</kp0>
+        <kp1>30.2</kp1>
+        <kp2>18.415</kp2> -->
+        <kp0>200.2</kp0>
+        <kp1>60.2</kp1>
+        <kp2>42.415</kp2>
+        <kd0>1</kd0>
+        <kd1>1.5</kd1>
+        <kd2>0.5</kd2>
+        <!--
+        <kp0>80</kp0>
+        <kp1>40</kp1>
+        <kp2>20</kp2>
+        <kd0>1</kd0>
+        <kd1>1</kd1>
+        <kd2>0.5</kd2> -->
+        <!--
+        <kp0>200</kp0>
+        <kp1>120</kp1>
+        <kp2>60</kp2>
+        <kd0>1</kd0>
+        <kd1>1</kd1>
+        <kd2>0.5</kd2> -->
+        <!-- adding higher gains for the swing leg -->
+        <kpsw0>300</kpsw0>
+        <kpsw1>300</kpsw1>
+        <kpsw2>300</kpsw2>
+        <kdsw0>6</kdsw0>
+        <kdsw1>6</kdsw1>
+        <kdsw2>6</kdsw2>
+       </plugin>
     </gazebo>
     <!-- IMU sensor -->
     <gazebo>
       <plugin name="imu_sensor" filename="libgazebo_ros_imu.so">
-          <alwaysOn>true</alwaysOn>
-          <bodyName>base</bodyName>
-          <frameName>base</frameName>
-          <topicName>/shvan/imu</topicName>
-          <serviceName>imu_service</serviceName>
-          <xyzOffset> 0 0 0 </xyzOffset>
-          <rpyOffset> 0 0 0 </rpyOffset>
-          <gaussianNoise>0.001</gaussianNoise>
-          <updateRate>1000.0</updateRate>
+        <alwaysOn>true</alw aysOn>
+        <bodyName>base</bodyName>
+        <frameName>base</frameName>
+        <topicName>/shvan/imu</topicName>
+        <serviceName>imu_service</serviceName>
+        <xyzOffset> 0 0 0 </xyzOffset>
+        <rpyOffset> 0 0 0 </rpyOffset>
+        <gaussianNoise>0.001</gaussianNoise>
+        <updateRate>1000.0</updateRate>
       </plugin>
   </gazebo>
@@ -164,5 +164,5 @@
     <!-- RR foot -->
     <gazebo reference="RH_FOOT">
-        <material>Gazebo/Black</material>
+      <material>Gazebo/Black</material>
       <collision>
         <surface>

File: legged_examples/legged_unitree/legged_unitree_description/urdf/common/leg_m2.xacro (robot description, xacro)
@@ -1,7 +1,7 @@
 <?xml version="1.0"?>
 <robot xmlns:xacro="http://www.ros.org/wiki/xacro">
-    <!-- <xacro:include filename="$(find m2_description)/xacro/transmission.xacro"/> -->
+    <xacro:include filename="$(find legged_unitree_description)/urdf/common/transmission.xacro"/>
     <xacro:include filename="$(find legged_unitree_description)/urdf/$(arg robot_type)/const.xacro"/>
-    <xacro:macro name="leg_m2" params="name mirror front_hind">
+    <xacro:macro name="leg_m2" params="name mirror front_hind ">
     <xacro:property name="STL_path" value="file://$(find legged_unitree_description)/meshes/m2"/>
         <!-- HAA_joint -->
@@ -196,4 +196,31 @@
             <disableFixedJointLumping>true</disableFixedJointLumping>
         </gazebo>
+        <gazebo reference="${name}_hip">
+            <mu1>0.2</mu1>
+            <mu2>0.2</mu2>
+            <material>svan_grey</material>
+        </gazebo>
+        <gazebo reference="${name}_thigh">
+            <mu1>0.2</mu1>
+            <mu2>0.2</mu2>
+            <self_collide>0</self_collide>
+            <material>svan_black</material>
+            <kp value="1000000.0"/>
+            <kd value="100.0"/>
+        </gazebo>
+        <gazebo reference="${name}_calf">
+            <mu1>0.6</mu1>
+            <mu2>0.6</mu2>
+            <self_collide>1</self_collide>
+        </gazebo>
+        <gazebo reference="${name}_FOOT">
+            <mu1>0.6</mu1>
+            <mu2>0.6</mu2>
+            <self_collide>1</self_collide>
+            <material>Gazebo/DarkGrey</material>
+            <kp value="1000000.0"/>
+            <kd value="100.0"/>
+        </gazebo>
+        <xacro:leg_transmission name="${name}"/>
      </xacro:macro>
 </robot>

File: legged_examples/legged_unitree/legged_unitree_description/urdf/common/transmission.xacro (robot description, xacro)
@@ -2,30 +2,30 @@
 <robot xmlns:xacro="http://www.ros.org/wiki/xacro">
     <xacro:macro name="leg_transmission" params="name">
-        <transmission name="${prefix}_HAA_tran">
+        <transmission name="${name}_HAA_tran">
             <type>transmission_interface/SimpleTransmission</type>
-            <joint name="${prefix}_HAA">
+            <joint name="${name}_HAA">
                 <hardwareInterface>hardware_interface/EffortJointInterface</hardwareInterface>
             </joint>
-            <actuator name="${prefix}_HAA_motor">
+            <actuator name="${name}_HAA_motor">
                 <hardwareInterface>hardware_interface/EffortJointInterface</hardwareInterface>
                 <mechanicalReduction>1</mechanicalReduction>
             </actuator>
         </transmission>
-        <transmission name="${prefix}_HFE_tran">
+        <transmission name="${name}_HFE_tran">
             <type>transmission_interface/SimpleTransmission</type>
-            <joint name="${prefix}_HFE">
+            <joint name="${name}_HFE">
                 <hardwareInterface>hardware_interface/EffortJointInterface</hardwareInterface>
             </joint>
-            <actuator name="${prefix}_HFE_motor">
+            <actuator name="${name}_HFE_motor">
                 <hardwareInterface>hardware_interface/EffortJointInterface</hardwareInterface>
                 <mechanicalReduction>1</mechanicalReduction>
             </actuator>
         </transmission>
-        <transmission name="${prefix}_KFE_tran">
+        <transmission name="${name}_KFE_tran">
             <type>transmission_interface/SimpleTransmission</type>
-            <joint name="${prefix}_KFE">
+            <joint name="${name}_KFE">
                 <hardwareInterface>hardware_interface/EffortJointInterface</hardwareInterface>
             </joint>
-            <actuator name="${prefix}_KFE_motor">
+            <actuator name="${name}_KFE_motor">
                 <hardwareInterface>hardware_interface/EffortJointInterface</hardwareInterface>
                 <mechanicalReduction>1</mechanicalReduction>

File: legged_examples/legged_unitree/legged_unitree_description/urdf/robot.xacro (robot description, xacro)
@@ -5,5 +5,5 @@
     <xacro:include filename="$(find legged_unitree_description)/urdf/common/leg.xacro"/>
     <xacro:include filename="$(find legged_unitree_description)/urdf/common/leg_m2.xacro"/>
-    <!-- <xacro:include filename="$(find legged_unitree_description)/urdf/common/gazebo.xacro"/> -->
+    <xacro:include filename="$(find legged_unitree_description)/urdf/common/gazebo.xacro"/>
     <xacro:include filename="$(find legged_unitree_description)/urdf/common/imu.xacro"/>
     <xacro:include filename="$(find legged_unitree_description)/urdf/$(arg robot_type)/const.xacro"/>
@@ -45,8 +45,8 @@
     <!-- leg xacro for m2  -->
     <xacro:if value="${'$(arg robot_type)' == 'm2'}">
-        <xacro:leg_m2 name="RF" mirror="1" front_hind="1"  />
-        <xacro:leg_m2 name="RH" mirror="1" front_hind="-1" />
-        <xacro:leg_m2 name="LH" mirror="-1"  front_hind="-1" />
-        <xacro:leg_m2 name="LF" mirror="-1"  front_hind="1"  />
+        <xacro:leg_m2 name="RF" mirror="1"  front_hind="1"  />
+        <xacro:leg_m2 name="RH" mirror="1"  front_hind="-1" />
+        <xacro:leg_m2 name="LH" mirror="-1" front_hind="-1" />
+        <xacro:leg_m2 name="LF" mirror="-1" front_hind="1"  />
     </xacro:if>
     <!-- leg xacro for other robots -->
@@ -65,4 +65,4 @@
         </xacro:leg>
     </xacro:if>
-    <xacro:include filename="$(find legged_unitree_description)/urdf/common/gazebo_m2.xacro"/>
+    <!-- <xacro:include filename="$(find legged_unitree_description)/urdf/common/gazebo_m2.xacro"/> -->
 </robot>

Commit message: fixed m2 joint config

File: legged_examples/legged_unitree/legged_unitree_description/urdf/common/gazebo_m2.xacro (robot description, xacro)
@@ -39,5 +39,5 @@
     <gazebo>
       <plugin name="imu_sensor" filename="libgazebo_ros_imu.so">
-        <alwaysOn>true</alw aysOn>
+        <alwaysOn>true</alwaysOn>
         <bodyName>base</bodyName>
         <frameName>base</frameName>

File: legged_examples/legged_unitree/legged_unitree_description/urdf/common/leg_m2.xacro (robot description, xacro)
@@ -64,5 +64,5 @@
         <!-- HFE -->
         <joint name="${name}_HFE" type="revolute">
-            <origin xyz="${front_hind*hip_j_com_x} ${mirror*hip_j_com_y} ${hip_j_com_z}" rpy="0 0 0" />
+            <origin xyz="${front_hind*hip_j_com_x} ${mirror*hip_j_com_y} ${hip_j_com_z}" rpy="0 1.57 0" />
             <parent link="${name}_hip"/>
             <child link="${name}_thigh"/>
@@ -111,5 +111,6 @@
         <!-- KFE -->
         <joint name="${name}_KFE" type="revolute">
-            <origin xyz="${front_hind*knee_j_com_x} ${mirror*knee_j_com_y} ${knee_j_com_z}" rpy="0 0 0" />
+        <!-- can't set the rotation higher than this,idk why (-Mehul) -->
+            <origin xyz="${front_hind*knee_j_com_x} ${mirror*knee_j_com_y} ${knee_j_com_z}" rpy="0 -1.5 0" />
             <parent link="${name}_thigh"/>
             <child link="${name}_calf"/>
@@ -196,5 +197,5 @@
             <disableFixedJointLumping>true</disableFixedJointLumping>
         </gazebo>
-        <gazebo reference="${name}_hip">
+        <!-- <gazebo reference="${name}_hip">
             <mu1>0.2</mu1>
             <mu2>0.2</mu2>
@@ -221,5 +222,5 @@
             <kp value="1000000.0"/>
             <kd value="100.0"/>
-        </gazebo>
+        </gazebo> -->
         <xacro:leg_transmission name="${name}"/>
      </xacro:macro>
