Commit message: reverted the changed of rotated axes on joints, robot now loads correctly; added default value for stance

File: legged_examples/legged_unitree/legged_unitree_description/urdf/common/gazebo.xacro (robot description, xacro)
@@ -21,3 +21,57 @@
         </plugin>
     </gazebo>
+    <!-- Foot contacts. -->
+      <!-- <gazebo>
+          <plugin name="contact_plugin" filename="libcontact_plugin_new.so">
+            <link1>foot_FR</link1>
+            <link2>FL_FOOT</link2>
+            <link3>RL_FOOT</link3>
+            <link4>RR_FOOT</link4>
+            <contact_model>0</contact_model>
+          </plugin>
+      </gazebo> -->
+      <!-- <gazebo reference="RF_FOOT">
+        <sensor name="FR_contact_sensor" type="contact">
+          <always_on>1</always_on>
+          <plugin name="contact_plugin_default" filename="libcontact_plugin_default.so">
+            <foot_link>FR</foot_link>
+          </plugin>
+          <contact>
+            <collision>foot_FR_collision</collision>
+          </contact>
+        </sensor>
+      </gazebo>
+      <gazebo reference="LF_FOOT">
+        <sensor name="FL_contact_sensor" type="contact">
+          <always_on>1</always_on>
+          <plugin name="contact_plugin_default" filename="libcontact_plugin_default.so">
+            <foot_link>FL</foot_link>
+          </plugin>
+          <contact>
+            <collision>FL_FOOT_collision</collision>
+          </contact>
+        </sensor>
+      </gazebo>
+      <gazebo reference="LH_FOOT">
+        <sensor name="RL_contact_sensor" type="contact">
+          <always_on>1</always_on>
+          <plugin name="contact_plugin_default" filename="libcontact_plugin_default.so">
+            <foot_link>RL</foot_link>
+          </plugin>
+          <contact>
+            <collision>RL_FOOT_collision</collision>
+          </contact>
+        </sensor>
+      </gazebo>
+      <gazebo reference="RH_FOOT">
+        <sensor name="RR_contact_sensor" type="contact">
+          <always_on>1</always_on>
+          <plugin name="contact_plugin_default" filename="libcontact_plugin_default.so">
+            <foot_link>RR</foot_link>
+          </plugin>
+          <contact>
+            <collision>RR_FOOT_collision</collision>
+          </contact>
+        </sensor>
+      </gazebo> -->
 </robot>

File: legged_examples/legged_unitree/legged_unitree_description/urdf/common/gazebo_m2.xacro (robot description, xacro)
@@ -27,5 +27,5 @@
         <kd1>1</kd1>
         <kd2>0.5</kd2> -->
-        <!-- adding higher gains for the swing leg -->
+        <!-- adding higher gains   for the swing leg -->
         <kpsw0>300</kpsw0>
         <kpsw1>300</kpsw1>

File: legged_examples/legged_unitree/legged_unitree_description/urdf/common/leg_m2.xacro (robot description, xacro)
@@ -64,5 +64,5 @@
         <!-- HFE -->
         <joint name="${name}_HFE" type="revolute">
-            <origin xyz="${front_hind*hip_j_com_x} ${mirror*hip_j_com_y} ${hip_j_com_z}" rpy="0 1.57 0" />
+            <origin xyz="${front_hind*hip_j_com_x} ${mirror*hip_j_com_y} ${hip_j_com_z}" rpy="0 0 0" />
             <parent link="${name}_hip"/>
             <child link="${name}_thigh"/>
@@ -111,6 +111,5 @@
         <!-- KFE -->
         <joint name="${name}_KFE" type="revolute">
-        <!-- can't set the rotation higher than this,idk why (-Mehul) -->
-            <origin xyz="${front_hind*knee_j_com_x} ${mirror*knee_j_com_y} ${knee_j_com_z}" rpy="0 -1.5 0" />
+            <origin xyz="${front_hind*knee_j_com_x} ${mirror*knee_j_com_y} ${knee_j_com_z}" rpy="0 0 0" />
             <parent link="${name}_thigh"/>
             <child link="${name}_calf"/>
@@ -197,5 +196,5 @@
             <disableFixedJointLumping>true</disableFixedJointLumping>
         </gazebo>
-        <!-- <gazebo reference="${name}_hip">
+        <gazebo reference="${name}_hip">
             <mu1>0.2</mu1>
             <mu2>0.2</mu2>
@@ -211,16 +210,17 @@
         </gazebo>
         <gazebo reference="${name}_calf">
-            <mu1>0.6</mu1>
-            <mu2>0.6</mu2>
+            <mu1>0.2</mu1>
+            <mu2>0.2</mu2>
             <self_collide>1</self_collide>
         </gazebo>
+        <!-- changing the values to 0.6 in this fricks up the model when loading. why? -->
         <gazebo reference="${name}_FOOT">
-            <mu1>0.6</mu1>
-            <mu2>0.6</mu2>
+            <mu1>0.2</mu1>
+            <mu2>0.2</mu2>
             <self_collide>1</self_collide>
             <material>Gazebo/DarkGrey</material>
             <kp value="1000000.0"/>
             <kd value="100.0"/>
-        </gazebo> -->
+        </gazebo>
         <xacro:leg_transmission name="${name}"/>
      </xacro:macro>
