Commit message: updated package legged_xterra_description

File: legged_examples/legged_xterra/legged_xterra_description/urdf/common/leg.xacro (robot description, xacro)
@@ -2,189 +2,194 @@
 <robot xmlns:xacro="http://www.ros.org/wiki/xacro">
     <xacro:include filename="$(find legged_xterra_description)/urdf/common/transmission.xacro"/>
-    <xacro:macro name="leg" params="prefix mesh_path mirror mirror_dae front_hind front_hind_dae *origin">
-        <joint name="${prefix}_HAA" type="revolute">
-            <xacro:insert_block name="origin"/>
-            <parent link="base"/>
-            <child link="${prefix}_hip"/>
-            <axis xyz="1 0 0"/>
-            <dynamics damping="${damping}" friction="${friction}"/>
-            <xacro:if value="${(mirror_dae == True)}">
-                <limit effort="${hip_torque_max}" velocity="${hip_velocity_max}" lower="${hip_position_min}"
-                       upper="${hip_position_max}"/>
-            </xacro:if>
-            <xacro:if value="${(mirror_dae == False)}">
-                <limit effort="${hip_torque_max}" velocity="${hip_velocity_max}" lower="${-hip_position_max}"
-                       upper="${-hip_position_min}"/>
-            </xacro:if>
-        </joint>
-        <link name="${prefix}_hip">
+    <xacro:macro name="leg" params="name mirror front_hind">
+    <xacro:property name="STL_path" value="file://$(find legged_xterra_description)/meshes/m2"/>
+        <!-- hip_link-->
+        <link name="${name}_hip_link">
+            <inertial>
+                <origin xyz="${front_hind*abd_l_com_x} ${mirror*abd_l_com_y} ${abd_l_com_z}"  rpy="0 0 0" />
+                <mass value="${abd_l_mass}"/>
+                <inertia
+                    ixx="${abd_l_ixx}" ixy="${mirror*front_hind*abd_l_ixy}" ixz="${front_hind*abd_l_ixz}"
+                    iyy="${abd_l_iyy}" iyz="${mirror*abd_l_iyz}"
+                    izz="${abd_l_izz}"/>
+            </inertial>
             <visual>
-                <xacro:if value="${(mirror_dae == True) and (front_hind_dae == True)}">
-                    <origin rpy="0 0 0" xyz="0 0 0"/>
+                <xacro:if value="${(front_hind == 1)}">
+                    <origin rpy="0 0 0" xyz="0 0 0" />
                 </xacro:if>
-                <xacro:if value="${(mirror_dae == False) and (front_hind_dae == True)}">
-                    <origin rpy="${pi} 0 0" xyz="0 0 0"/>
-                </xacro:if>
-                <xacro:if value="${(mirror_dae == True) and (front_hind_dae == False)}">
-                    <origin rpy="0 ${pi} 0" xyz="0 0 0"/>
-                </xacro:if>
-                <xacro:if value="${(mirror_dae == False) and (front_hind_dae == False)}">
-                    <origin rpy="${pi} ${pi} 0" xyz="0 0 0"/>
+                <xacro:if value="${(front_hind == -1)}">
+                    <origin rpy="${PI} ${PI} 0" xyz="0 0 0"/>
                 </xacro:if>
                 <geometry>
-                    <mesh filename="${mesh_path}/hip.dae"
-                          scale="1 1 1"/>
+                    <xacro:if value="${(mirror == 1 and front_hind == 1) or (mirror == -1 and front_hind == -1)}">
+                        <mesh filename="${STL_path}/FR_hip.STL" />
+                    </xacro:if>
+                    <xacro:if value="${(mirror == -1 and front_hind == 1) or (mirror == 1 and front_hind == -1)}">
+                        <mesh filename="${STL_path}/FL_hip.STL" />
+                    </xacro:if>
                 </geometry>
-                <material name="orange"/>
+                <material name = "svan_grey"/>
             </visual>
             <collision>
-                <origin rpy="${pi/2.0} 0 0" xyz="0 0 0"/>
+                <xacro:if value="${(front_hind == 1)}">
+                    <origin rpy="0 0 0" xyz="0 0 0" />
+                </xacro:if>
+                <xacro:if value="${(front_hind == -1)}">
+                    <origin rpy="${PI} ${PI} 0" xyz="0 0 0"/>
+                </xacro:if>
                 <geometry>
-                    <cylinder length="${hip_length}" radius="${hip_radius}"/>
+                    <xacro:if value="${(mirror == 1 and front_hind == 1) or (mirror == -1 and front_hind == -1)}">
+                        <mesh filename="${STL_path}/FR_hip.STL" />
+                    </xacro:if>
+                    <xacro:if value="${(mirror == -1 and front_hind == 1) or (mirror == 1 and front_hind == -1)}">
+                        <mesh filename="${STL_path}/FL_hip.STL" />
+                    </xacro:if>
                 </geometry>
             </collision>
+        </link>
+        <!-- HAA_joint -->
+        <joint name="${name}_HAA_joint" type="revolute">
+            <origin xyz="${front_hind*abd_j_com_x} ${mirror*abd_j_com_y} ${abd_j_com_z}" rpy="0 0 0" />
+            <parent link="base"/>
+            <child link="${name}_hip_link"/>
+            <xacro:if value="${(front_hind == 1)}">
+                <axis xyz="1 0 0"/>
+            </xacro:if>
+            <xacro:if value="${(front_hind == -1)}">
+                <axis xyz="-1 0 0"/>
+            </xacro:if>
+            <limit lower="${abd_j_lower}" upper="${abd_j_upper}" effort="${abd_j_effort}" velocity="${abd_j_velocity}"/>
+        </joint>
+        <!-- thigh link -->
+        <link name="${name}_thigh_link">
             <inertial>
-                <origin rpy="0 0 0" xyz="${hip_com_x*front_hind} ${hip_com_y*mirror} ${hip_com_z}"/>
-                <mass value="${hip_mass}"/>
+                <origin xyz="${front_hind*hip_l_com_x} ${-mirror*hip_l_com_y} ${hip_l_com_z}"  rpy="0 0 0" />
+                <mass value="${hip_l_mass}"/>
                 <inertia
-                        ixx="${hip_ixx}" ixy="${hip_ixy*mirror*front_hind}" ixz="${hip_ixz*front_hind}"
-                        iyy="${hip_iyy}" iyz="${hip_iyz*mirror}"
-                        izz="${hip_izz}"/>
+                    ixx="${hip_l_ixx}" ixy="${mirror*front_hind*hip_l_ixy}" ixz="${front_hind*hip_l_ixz}"
+                    iyy="${hip_l_iyy}" iyz="${mirror*hip_l_iyz}"
+                    izz="${hip_l_izz}"/>
             </inertial>
-        </link>
-        <joint name="${prefix}_HFE" type="revolute">
-            <origin rpy="0 0 0" xyz="0 ${thigh_offset*mirror} 0"/>
-            <parent link="${prefix}_hip"/>
-            <child link="${prefix}_thigh"/>
-            <axis xyz="0 1 0"/>
-            <dynamics damping="${damping}" friction="${friction}"/>
-            <limit effort="${thigh_torque_max}" velocity="${thigh_velocity_max}" lower="${thigh_position_min}"
-                   upper="${thigh_position_max}"/>
-        </joint>
-        <link name="${prefix}_thigh">
             <visual>
                 <origin rpy="0 0 0" xyz="0 0 0"/>
                 <geometry>
-                    <xacro:if value="${mirror_dae == True}">
-                        <mesh filename="${mesh_path}/FL_thigh.stl"
-                              scale="1 1 1"/>
+                    <xacro:if value="${mirror == 1}">
+                        <mesh filename="${STL_path}/FR_thigh.STL" />
                     </xacro:if>
-                    <xacro:if value="${mirror_dae == False}">
-                        <mesh filename="${mesh_path}/FL_thigh.stl"
-                              scale="1 1 1"/>
+                    <xacro:if value="${mirror == -1}">
+                        <mesh filename="${STL_path}/FL_thigh.STL" />
                     </xacro:if>
                 </geometry>
-                <material name="orange"/>
-            </visual>
-            <collision>
-                <origin rpy="0 ${pi/2.0+0.1} 0" xyz="${thigh_x_offset} 0 ${-thigh_length/2.0}"/>
-                <geometry>
-                    <box size="${thigh_length} ${thigh_width} ${thigh_height}"/>
-                </geometry>
-            </collision>
-            <collision>
-                <origin rpy="${pi/2.0} 0 0" xyz="0 ${mirror*thigh_shoulder_y_offset} 0"/>
-                <geometry>
-                    <cylinder length="${thigh_shoulder_length}" radius="${thigh_shoulder_radius}"/>
-                </geometry>
-            </collision>
-            <inertial>
-                <origin rpy="0 0 0" xyz="${thigh_com_x} ${thigh_com_y*mirror} ${thigh_com_z}"/>
-                <mass value="${thigh_mass}"/>
-                <inertia
-                        ixx="${thigh_ixx}" ixy="${thigh_ixy*mirror}" ixz="${thigh_ixz}"
-                        iyy="${thigh_iyy}" iyz="${thigh_iyz*mirror}"
-                        izz="${thigh_izz}"/>
-            </inertial>
-        </link>
-        <joint name="${prefix}_KFE" type="revolute">
-            <origin rpy="0 0 0" xyz="0 0 ${-thigh_length}"/>
-            <parent link="${prefix}_thigh"/>
-            <child link="${prefix}_calf"/>
-            <axis xyz="0 1 0"/>
-            <dynamics damping="${damping}" friction="${friction}"/>
-            <limit effort="${calf_torque_max}" velocity="${calf_velocity_max}" lower="${calf_position_min}" upper="${calf_position_max}"/>
-        </joint>
-        <link name="${prefix}_calf">
-            <visual>
-                <origin rpy="0 0 0" xyz="0 0 0"/>
-                <geometry>
-                    <mesh filename="${mesh_path}/calf.dae"
-                          scale="1 1 1"/>
-                </geometry>
-                <material name="orange"/>
-            </visual>
-            <collision>
-                <origin rpy="0 ${pi/2.0} 0" xyz="${calf_x_offset} 0 ${-calf_length/2.0}"/>
-                <geometry>
-                    <box size="${calf_length} ${calf_width} ${calf_height}"/>
-                </geometry>
-            </collision>
-            <inertial>
-                <origin rpy="0 0 0" xyz="${calf_com_x} ${calf_com_y} ${calf_com_z}"/>
-                <mass value="${calf_mass}"/>
-                <inertia
-                        ixx="${calf_ixx}" ixy="${calf_ixy}" ixz="${calf_ixz}"
-                        iyy="${calf_iyy}" iyz="${calf_iyz}"
-                        izz="${calf_izz}"/>
-            </inertial>
-        </link>
-        <joint name="${prefix}_foot_fixed" type="fixed" dont_collapse="true">
-            <origin rpy="0 0 0" xyz="0 0 ${-(calf_length)}"/>
-            <parent link="${prefix}_calf"/>
-            <child link="${prefix}_FOOT"/>
-        </joint>
-        <link name="${prefix}_FOOT">
-            <visual>
-                <origin rpy="0 0 0" xyz="0 0 0"/>
-                <geometry>
-                    <sphere radius="${foot_radius-0.01}"/>
-                </geometry>
-                <material name="orange"/>
+                <material name = "svan_black"/>
             </visual>
             <collision>
                 <origin rpy="0 0 0" xyz="0 0 0"/>
                 <geometry>
-                    <sphere radius="${foot_radius}"/>
+                    <xacro:if value="${mirror == 1}">
+                        <mesh filename="${STL_path}/FR_thigh.STL" />
+                    </xacro:if>
+                    <xacro:if value="${mirror == -1}">
+                        <mesh filename="${STL_path}/FL_thigh.STL" />
+                    </xacro:if>
                 </geometry>
             </collision>
+        </link>
+        <!-- HFE_joint -->
+        <joint name="${name}_HFE_joint" type="revolute">
+            <origin xyz="${front_hind*hip_j_com_x} ${mirror*hip_j_com_y} ${hip_j_com_z}" rpy="0 0 0" />
+            <parent link="${name}_hip_link"/>
+            <child link="${name}_thigh_link"/>
+            <xacro:if value="${(mirror == 1)}">
+                <axis xyz="0 1 0"/>
+            </xacro:if>
+            <xacro:if value="${(mirror == -1)}">
+                <axis xyz="0 1 0"/>
+            </xacro:if>
+            <limit lower="${hip_j_lower}" upper="${hip_j_upper}" effort="${hip_j_effort}" velocity="${hip_j_velocity}"/>
+        </joint>
+        <!-- shank_link-->
+        <link name="${name}_shank_link">
             <inertial>
-                <mass value="${foot_mass}"/>
+                <origin xyz="${front_hind*knee_l_com_x} ${mirror*knee_l_com_y} ${knee_l_com_z}"  rpy="0 0 0" />
+                <mass value="${knee_l_mass}"/>
                 <inertia
-                        ixx="${(2*foot_mass)/5.0*(foot_radius*foot_radius)}" ixy="0.0" ixz="0.0"
-                        iyy="${(2*foot_mass)/5.0*(foot_radius*foot_radius)}" iyz="0.0"
-                        izz="${(2*foot_mass)/5.0*(foot_radius*foot_radius)}"/>
+                    ixx="${knee_l_ixx}" ixy="${mirror*knee_l_ixy}" ixz="${knee_l_ixz}"
+                    iyy="${knee_l_iyy}" iyz="${mirror*knee_l_iyz}"
+                    izz="${knee_l_izz}"/>
             </inertial>
+            <visual>
+                <origin rpy="0 0 0" xyz="0 0 0"/>
+                <geometry>
+                    <xacro:if value="${mirror == 1}">
+                        <mesh filename="${STL_path}/FR_shank.STL" />
+                    </xacro:if>
+                    <xacro:if value="${mirror == -1}">
+                        <mesh filename="${STL_path}/FL_shank.STL" />
+                    </xacro:if>
+                </geometry>
+                <material name = "svan_black"/>
+            </visual>
+            <collision>
+                <origin rpy="0 0 0" xyz="0 0 0"/>
+                <geometry>
+                    <xacro:if value="${mirror == 1}">
+                        <mesh filename="${STL_path}/FR_shank.STL" />
+                    </xacro:if>
+                    <xacro:if value="${mirror == -1}">
+                        <mesh filename="${STL_path}/FL_shank.STL" />
+                    </xacro:if>
+                </geometry>
+            </collision>
         </link>
-        <gazebo reference="${prefix}_foot_fixed">
-            <disableFixedJointLumping>true</disableFixedJointLumping>
-        </gazebo>
-        <gazebo reference="${prefix}_hip">
-            <mu1>0.2</mu1>
-            <mu2>0.2</mu2>
-            <material>Gazebo/DarkGrey</material>
-        </gazebo>
-        <gazebo reference="${prefix}_thigh">
-            <mu1>0.2</mu1>
-            <mu2>0.2</mu2>
-            <self_collide>0</self_collide>
-            <material>Gazebo/DarkGrey</material>
-            <kp value="1000000.0"/>
-            <kd value="100.0"/>
-        </gazebo>
-        <gazebo reference="${prefix}_calf">
-            <mu1>0.6</mu1>
-            <mu2>0.6</mu2>
-            <self_collide>1</self_collide>
-        </gazebo>
-        <gazebo reference="${prefix}_FOOT">
-            <mu1>0.6</mu1>
-            <mu2>0.6</mu2>
-            <self_collide>1</self_collide>
-            <material>Gazebo/DarkGrey</material>
-            <kp value="1000000.0"/>
-            <kd value="100.0"/>
-        </gazebo>
-        <xacro:leg_transmission name="${prefix}"/>
-    </xacro:macro>
+        <!-- KFE_joint -->
+        <joint name="${name}_KFE_joint" type="revolute">
+            <origin xyz="${front_hind*knee_j_com_x} ${mirror*knee_j_com_y} ${knee_j_com_z}" rpy="0 0 0" />
+            <parent link="${name}_thigh_link"/>
+            <child link="${name}_shank_link"/>
+            <xacro:if value="${(mirror == 1)}">
+                <axis xyz="0 1 0"/>
+            </xacro:if>
+            <xacro:if value="${(mirror == -1)}">
+                <axis xyz="0 1 0"/>
+            </xacro:if>
+            <limit lower="${knee_j_lower}" upper="${knee_j_upper}" effort="${knee_j_effort}" velocity="${knee_j_velocity}"/>
+        </joint>
+        <!-- foot-->
+        <link name="foot_${name}">
+            <contact>
+                <friction_anchor/>
+                <stiffness value="${foot_stiffness}"/>
+                <damping value="${foot_damping}"/>
+                <spinning_friction value="${foot_spinning_friction}"/>
+                <lateral_friction value="${foot_lateral_friction}"/>
+            </contact>
+            <inertial>
+                <origin xyz="${front_hind*foot_l_com_x} ${mirror*foot_l_com_y} ${foot_l_com_z}"  rpy="0 0 0" />
+                <mass value="${foot_l_mass}"/>
+                <inertia
+                    ixx="${foot_l_ixx}" ixy="${mirror*front_hind*foot_l_ixy}" ixz="${front_hind*foot_l_ixz}"
+                    iyy="${foot_l_iyy}" iyz="${mirror*foot_l_iyz}"
+                    izz="${foot_l_izz}"/>
+            </inertial>
+            <visual>
+            <geometry>
+                 <mesh filename="${STL_path}/FL_foot.STL" />
+            </geometry>
+            </visual>
+            <collision>
+            <geometry>
+                <mesh filename="${STL_path}/FL_foot.STL" />
+            </geometry>
+            </collision>
+        </link>
+        <!-- foot_j -->
+        <joint name="${name}_foot_j" type="revolute">
+            <origin xyz="${foot_j_com_x} ${mirror*foot_j_com_y} ${foot_j_com_z}" rpy="0 0 0" />
+            <parent link="${name}_shank_link"/>
+            <child link="foot_${name}"/>
+            <axis xyz="0 0 1"/>
+            <limit lower="0" upper="0" effort="1000" velocity="0" />
+        </joint>
+        <xacro:leg_transmission name="${name}"/>
+     </xacro:macro>
 </robot>

File: legged_examples/legged_xterra/legged_xterra_description/urdf/common/transmission.xacro (robot description, xacro)
@@ -4,5 +4,5 @@
         <transmission name="${name}_HAA_tran">
             <type>transmission_interface/SimpleTransmission</type>
-            <joint name="${name}_HAA">
+            <joint name="${name}_HAA_joint">
                 <hardwareInterface>hardware_interface/EffortJointInterface</hardwareInterface>
             </joint>
@@ -14,5 +14,5 @@
         <transmission name="${name}_HFE_tran">
             <type>transmission_interface/SimpleTransmission</type>
-            <joint name="${name}_HFE">
+            <joint name="${name}_HFE_joint">
                 <hardwareInterface>hardware_interface/EffortJointInterface</hardwareInterface>
             </joint>
@@ -24,5 +24,5 @@
         <transmission name="${name}_KFE_tran">
             <type>transmission_interface/SimpleTransmission</type>
-            <joint name="${name}_KFE">
+            <joint name="${name}_KFE_joint">
                 <hardwareInterface>hardware_interface/EffortJointInterface</hardwareInterface>
             </joint>
