Commit message: updated package legged_xterra_description

File: legged_examples/legged_xterra/legged_xterra_description/urdf/m2/const.xacro (robot description, xacro)
@@ -1,107 +1,120 @@
 <?xml version="1.0"?>
-<robot xmlns:xacro="http://www.ros.org/wiki/xacro" name="m2_description">
-    <!-- Constants for robot dimensions -->
-    <xacro:property name="PI" value="3.1415926535897931"/>
-    <xacro:property name="stick_mass" value="0.00001"/>
-    <!-- simplified collision value -->
-    <xacro:property name="trunk_width" value="0.0935"/>
-    <xacro:property name="trunk_length" value="0.3762"/>
-    <xacro:property name="trunk_height" value="0.114"/>
-    <xacro:property name="hip_radius" value="0.046"/>
-    <xacro:property name="hip_length" value="0.04"/>
-    <xacro:property name="thigh_shoulder_radius" value="0.041"/>
-    <xacro:property name="thigh_shoulder_length" value="0.032"/>
-    <xacro:property name="thigh_shoulder_y_offset" value="0.0465"/>
-    <xacro:property name="thigh_shoulder_x_offset" value="0.1934"/>
-    <xacro:property name="thigh_width" value="0.0245"/>
-    <xacro:property name="thigh_height" value="0.034"/>
-    <xacro:property name="thigh_x_offset" value="-0.0"/>
-    <xacro:property name="thigh_y_offset" value="-0.0955"/>
-    <xacro:property name="calf_width" value="0.016"/>
-    <xacro:property name="calf_height" value="0.016"/>
-    <xacro:property name="calf_x_offset" value="0.0"/>
-    <xacro:property name="foot_radius" value="0.02"/>
-    <xacro:property name="stick_radius" value="0.01"/>
-    <xacro:property name="stick_length" value="0.2"/>
-    <!-- kinematic value -->
-    <xacro:property name="thigh_offset" value="0.0955"/>
-    <xacro:property name="thigh_length" value="0.213"/>
-    <xacro:property name="calf_length" value="0.213"/>
-    <!-- leg offset from trunk center value -->
-    <xacro:property name="leg_offset_x" value="0.1934"/>
-    <xacro:property name="leg_offset_y" value="0.0465"/>
-    <xacro:property name="trunk_offset_z" value="0.01675"/>
-    <xacro:property name="hip_offset" value="0.0955"/>
-    <!-- offset of link locations (left front) -->
-    <xacro:property name="hip_offset_x" value="0.1934"/>
-    <xacro:property name="hip_offset_y" value="0.0465"/>
-    <xacro:property name="hip_offset_z" value="0.0"/>
-    <xacro:property name="thigh_offset_x" value="0"/>
-    <xacro:property name="thigh_offset_y" value="0.0955"/>
-    <xacro:property name="thigh_offset_z" value="0.0"/>
-    <xacro:property name="calf_offset_x" value="0.0"/>
-    <xacro:property name="calf_offset_y" value="0.0"/>
-    <xacro:property name="calf_offset_z" value="-0.213"/>
-    <!-- joint limits -->
-    <xacro:property name="damping" value="0.0"/>
-    <xacro:property name="friction" value="0.0"/>
-    <xacro:property name="hip_position_max" value="1.0472"/>
-    <xacro:property name="hip_position_min" value="-1.0472"/>
-    <xacro:property name="hip_velocity_max" value="30.1"/>
-    <xacro:property name="hip_torque_max" value="23.7"/>
-    <xacro:property name="thigh_position_max" value="3.4907"/>
-    <xacro:property name="thigh_position_min" value="-1.5708"/>
-    <xacro:property name="thigh_velocity_max" value="30.1"/>
-    <xacro:property name="thigh_torque_max" value="23.7"/>
-    <xacro:property name="calf_position_max" value="-0.83776"/>
-    <xacro:property name="calf_position_min" value="-2.7227"/>
-    <xacro:property name="calf_velocity_max" value="20.06"/>
-    <xacro:property name="calf_torque_max" value="35.55"/>
-    <!-- dynamics inertial value -->
-    <!-- trunk -->
-    <xacro:property name="trunk_mass" value="6.921"/>
-    <xacro:property name="trunk_com_x" value="0.021112"/>
-    <xacro:property name="trunk_com_y" value="0.00"/>
-    <xacro:property name="trunk_com_z" value="-0.005366"/>
-    <xacro:property name="trunk_ixx" value="0.02448"/>
-    <xacro:property name="trunk_ixy" value="0.00012166"/>
-    <xacro:property name="trunk_ixz" value="0.0014849"/>
-    <xacro:property name="trunk_iyy" value="0.098077"/>
-    <xacro:property name="trunk_iyz" value="-3.12E-05"/>
-    <xacro:property name="trunk_izz" value="0.107"/>
-    <!-- hip (left front) -->
-    <xacro:property name="hip_mass" value="0.678"/>
-    <xacro:property name="hip_com_x" value="-0.0054"/>
-    <xacro:property name="hip_com_y" value="0.00194"/>
-    <xacro:property name="hip_com_z" value="-0.000105"/>
-    <xacro:property name="hip_ixx" value="0.00048"/>
-    <xacro:property name="hip_ixy" value="-3.01E-06"/>
-    <xacro:property name="hip_ixz" value="1.11E-06"/>
-    <xacro:property name="hip_iyy" value="0.000884"/>
-    <xacro:property name="hip_iyz" value="-1.42E-06"/>
-    <xacro:property name="hip_izz" value="0.000596"/>
-    <!-- thigh -->
-    <xacro:property name="thigh_mass" value="1.152"/>
-    <xacro:property name="thigh_com_x" value="-0.00374"/>
-    <xacro:property name="thigh_com_y" value="-0.0223"/>
-    <xacro:property name="thigh_com_z" value="-0.0327"/>
-    <xacro:property name="thigh_ixx" value="0.00584"/>
-    <xacro:property name="thigh_ixy" value="8.72E-05"/>
-    <xacro:property name="thigh_ixz" value="-0.000289"/>
-    <xacro:property name="thigh_iyy" value="0.0058"/>
-    <xacro:property name="thigh_iyz" value="0.000808"/>
-    <xacro:property name="thigh_izz" value="0.00103"/>
-    <!-- calf -->
-    <xacro:property name="calf_mass" value="0.154"/>
-    <xacro:property name="calf_com_x" value="0.00548"/>
-    <xacro:property name="calf_com_y" value="-0.000975"/>
-    <xacro:property name="calf_com_z" value="-0.115"/>
-    <xacro:property name="calf_ixx" value="0.00108"/>
-    <xacro:property name="calf_ixy" value="3.4E-07"/>
-    <xacro:property name="calf_ixz" value="1.72E-05"/>
-    <xacro:property name="calf_iyy" value="0.0011"/>
-    <xacro:property name="calf_iyz" value="8.28E-06"/>
-    <xacro:property name="calf_izz" value="3.29E-05"/>
-    <!-- foot -->
-    <xacro:property name="foot_mass" value="0.06"/>
+<robot xmlns:xacro="http://www.ros.org/wiki/xacro">
+<xacro:property name="PI" value="3.14159265359"/>
+<!-- base -->
+<!-- <xacro:property name="base_com_x" value="0.002585"/>
+<xacro:property name="base_com_y" value="0.003221"/>
+<xacro:property name="base_com_z" value="0.008796"/>
+<xacro:property name="base_mass" value="5.428590"/>
+<xacro:property name="base_ixx" value="0.028959"/>
+<xacro:property name="base_ixy" value="-0.000021"/>
+<xacro:property name="base_ixz" value="0.001591"/>
+<xacro:property name="base_iyy" value="0.0601762"/>
+<xacro:property name="base_iyz" value="0.000025"/>
+<xacro:property name="base_izz" value="0.068516"/> -->
+<!-- without camera mount
+<xacro:property name="base_com_x" value="-0.002656"/>
+<xacro:property name="base_com_y" value="0.003430"/>
+<xacro:property name="base_com_z" value="0.000860"/>
+<xacro:property name="base_mass" value="5.016234"/>
+<xacro:property name="base_ixx" value="0.023890"/>
+<xacro:property name="base_ixy" value="-0.000506"/>
+<xacro:property name="base_ixz" value="-0.001154"/>
+<xacro:property name="base_iyy" value="0.053100"/>
+<xacro:property name="base_iyz" value="-0.000013"/>
+<xacro:property name="base_izz" value="0.065972"/> -->
+Here are the updated xacro properties based on the provided data:
+```xml
+<!-- base -->
+<xacro:property name="base_mass" value="5.18596663"/>
+<xacro:property name="base_com_x" value="0.00918208"/>
+<xacro:property name="base_com_y" value="-0.00133606"/>
+<xacro:property name="base_com_z" value="-0.00430117"/>
+<xacro:property name="base_ixx" value="0.02220107"/>
+<xacro:property name="base_ixy" value="-0.00019966"/>
+<xacro:property name="base_ixz" value="-0.00048929"/>
+<xacro:property name="base_iyy" value="0.05026338"/>
+<xacro:property name="base_iyz" value="-0.00001273"/>
+<xacro:property name="base_izz" value="0.06413613"/>
+<!-- abd FR-->
+<xacro:property name="abd_l_mass" value="1.12704463"/>
+<xacro:property name="abd_l_com_x" value="0.04244851"/>
+<xacro:property name="abd_l_com_y" value="-0.07733848"/>
+<xacro:property name="abd_l_com_z" value="0.00084768"/>
+<xacro:property name="abd_l_ixx" value="0.0026019"/>
+<xacro:property name="abd_l_ixy" value="0.0001226"/>
+<xacro:property name="abd_l_ixz" value="0.0000075"/>
+<xacro:property name="abd_l_iyy" value="0.0009202"/>
+<xacro:property name="abd_l_iyz" value="-0.0000024"/>
+<xacro:property name="abd_l_izz" value="0.0026365"/>
+<!-- hip FR -->
+<xacro:property name="hip_l_mass" value="0.15396568"/>
+<xacro:property name="hip_l_com_x" value="0.00000000"/>
+<xacro:property name="hip_l_com_y" value="-0.00262472"/>
+<xacro:property name="hip_l_com_z" value="-0.06933846"/>
+<xacro:property name="hip_l_ixx" value="0.00075104"/>
+<xacro:property name="hip_l_ixy" value="0.00000000"/>
+<xacro:property name="hip_l_ixz" value="0.00000000"/>
+<xacro:property name="hip_l_iyy" value="0.00076325"/>
+<xacro:property name="hip_l_iyz" value="-0.00002968"/>
+<xacro:property name="hip_l_izz" value="0.00004729"/>
+<!-- knee FR -->
+<xacro:property name="knee_l_mass" value="0.1244820"/>
+<xacro:property name="knee_l_com_x" value="-0.0010600"/>
+<xacro:property name="knee_l_com_y" value="0.0000090"/>
+<xacro:property name="knee_l_com_z" value="-0.0450013"/>
+<xacro:property name="knee_l_ixx" value="0.0005021"/>
+<xacro:property name="knee_l_ixy" value="0.0000000"/>
+<xacro:property name="knee_l_ixz" value="-0.0000127"/>
+<xacro:property name="knee_l_iyy" value="0.0005174"/>
+<xacro:property name="knee_l_iyz" value="0.0000001"/>
+<xacro:property name="knee_l_izz" value="0.0000202"/>
+<!-- foot FR-->
+<xacro:property name="foot_l_mass" value="0.02330447"/>
+<xacro:property name="foot_l_com_x" value="-0.00255660"/>
+<xacro:property name="foot_l_com_y" value="0.00017773"/>
+<xacro:property name="foot_l_com_z" value="-0.00416818"/>
+<xacro:property name="foot_l_ixx" value="0.00000262"/>
+<xacro:property name="foot_l_ixy" value="0.00000001"/>
+<xacro:property name="foot_l_ixz" value="-0.00000037"/>
+<xacro:property name="foot_l_iyy" value="0.00000262"/>
+<xacro:property name="foot_l_iyz" value="0.00000002"/>
+<xacro:property name="foot_l_izz" value="0.00000300"/>
+```
+<xacro:property name="foot_stiffness" value="30000"/>
+<xacro:property name="foot_damping" value="750"/>
+<xacro:property name="foot_spinning_friction" value="0.3"/>
+<xacro:property name="foot_lateral_friction" value="50"/>
+<!-- fr_abd_j -->
+<xacro:property name="abd_j_com_x" value="0.147"/>
+<xacro:property name="abd_j_com_y" value="-0.06"/>
+<xacro:property name="abd_j_com_z" value="0.00025"/>
+<xacro:property name="abd_j_axis" value="1 0 0"/>
+<xacro:property name="abd_j_lower" value="-4.8"/>
+<xacro:property name="abd_j_upper" value="4.8"/>
+<xacro:property name="abd_j_effort" value="20"/>
+<xacro:property name="abd_j_velocity" value="52.4"/>
+<!-- fr_hip_j -->
+<xacro:property name="hip_j_com_x" value="0.043751"/>
+<xacro:property name="hip_j_com_y" value="-0.08110"/>
+<xacro:property name="hip_j_com_z" value="0"/>
+<xacro:property name="hip_j_axis" value="0 -1 0"/>
+<xacro:property name="hip_j_effort" value="55"/>
+<xacro:property name="hip_j_lower" value="-4.047197551"/>
+<xacro:property name="hip_j_upper" value="4.188790205"/>
+<xacro:property name="hip_j_velocity" value="28.6"/>
+<!-- fr_knee_j -->
+<xacro:property name="knee_j_com_x" value="0"/>
+<xacro:property name="knee_j_com_y" value="0"/>
+<xacro:property name="knee_j_com_z" value="-0.1915"/>
+<xacro:property name="knee_j_axis" value="0 -1 0"/>
+<xacro:property name="knee_j_effort" value="55"/>
+<xacro:property name="knee_j_lower" value="-4.696533694"/>
+<xacro:property name="knee_j_upper" value="4.916297857"/>
+<xacro:property name="knee_j_velocity" value ="28.6"/>
+<!-- foot_j -->
+<xacro:property name="foot_j_com_x" value="-0.00351"/>
+<xacro:property name="foot_j_com_y" value="0"/>
+<xacro:property name="foot_j_com_z" value="-0.1901"/>
+<xacro:property name="foot_j_axis" value="0 0 1"/>
 </robot>

File: legged_examples/legged_xterra/legged_xterra_description/urdf/robot.xacro (robot description, xacro)
@@ -8,10 +8,10 @@
     <xacro:include filename="$(find legged_xterra_description)/urdf/$(arg robot_type)/const.xacro"/>
 <!--    <xacro:property name="mesh_path" value="../meshes"/>-->
-    <xacro:property name="mesh_path" value="$(find legged_xterra_description)/meshes/$(arg robot_type)"/>
+    <xacro:property name="mesh_path" value="file://$(find legged_xterra_description)/meshes/$(arg robot_type)"/>
     <link name="base">
         <visual>
             <origin rpy="0 0 0" xyz="0 0 0"/>
             <geometry>
-                <mesh filename="${mesh_path}/torso.stl" scale="1 1 1"/>
+                <mesh filename="${mesh_path}/torso.STL" scale="1 1 1"/>
             </geometry>
         </visual>
@@ -19,28 +19,20 @@
             <origin rpy="0 0 0" xyz="0 0 0"/>
             <geometry>
-                <box size="${trunk_length} ${trunk_width} ${trunk_height}"/>
+                <mesh filename="${mesh_path}/torso.STL" scale="1 1 1"/>
             </geometry>
         </collision>
         <inertial>
-            <origin rpy="0 0 0" xyz="${trunk_com_x} ${trunk_com_y} ${trunk_com_z}"/>
-            <mass value="${trunk_mass}"/>
+            <origin rpy="0 0 0" xyz="${base_com_x} ${base_com_y} ${base_com_z}"/>
+            <mass value="${base_mass}"/>
             <inertia
-                    ixx="${trunk_ixx}" ixy="${trunk_ixy}" ixz="${trunk_ixz}"
-                    iyy="${trunk_iyy}" iyz="${trunk_iyz}"
-                    izz="${trunk_izz}"/>
+                    ixx="${base_ixx}" ixy="${base_ixy}" ixz="${base_ixz}"
+                    iyy="${base_iyy}" iyz="${base_iyz}"
+                    izz="${base_izz}"/>
         </inertial>
     </link>
     <xacro:IMU connected_to="base" imu_name="base_imu" xyz="0. 0. 0." rpy="0. 0. 0."/>
-    <xacro:leg prefix="LF" mesh_path="${mesh_path}" mirror="1" mirror_dae="True" front_hind="1" front_hind_dae="True">
-        <origin rpy="0 0 0" xyz="${leg_offset_x} ${leg_offset_y} 0"/>
-    </xacro:leg>
-    <xacro:leg prefix="LH" mesh_path="${mesh_path}" mirror="1" mirror_dae="True" front_hind="-1" front_hind_dae="False">
-        <origin rpy="0 0 0" xyz="${-leg_offset_x} ${leg_offset_y} 0"/>
-    </xacro:leg>
-    <xacro:leg prefix="RF" mesh_path="${mesh_path}" mirror="-1" mirror_dae="False" front_hind="1" front_hind_dae="True">
-        <origin rpy="0 0 0" xyz="${leg_offset_x} ${-leg_offset_y} 0"/>
-    </xacro:leg>
-    <xacro:leg prefix="RH" mesh_path="${mesh_path}" mirror="-1" mirror_dae="False" front_hind="-1" front_hind_dae="False">
-        <origin rpy="0 0 0" xyz="${-leg_offset_x} ${-leg_offset_y} 0"/>
-    </xacro:leg>
+    <xacro:leg name="FR" mirror="1" front_hind="1"  />
+    <xacro:leg name="FL" mirror="-1"  front_hind="1"  />
+    <xacro:leg name="RR" mirror="1" front_hind="-1" />
+    <xacro:leg name="RL" mirror="-1"  front_hind="-1" />
 </robot>

Commit message: Changed joint names

File: legged_examples/legged_xterra/legged_xterra_description/urdf/common/leg.xacro (robot description, xacro)
@@ -49,5 +49,5 @@
         </link>
         <!-- HAA_joint -->
-        <joint name="${name}_HAA_joint" type="revolute">
+        <joint name="${name}_HAA" type="revolute">
             <origin xyz="${front_hind*abd_j_com_x} ${mirror*abd_j_com_y} ${abd_j_com_z}" rpy="0 0 0" />
             <parent link="base"/>
@@ -96,5 +96,5 @@
         </link>
         <!-- HFE_joint -->
-        <joint name="${name}_HFE_joint" type="revolute">
+        <joint name="${name}_HFE" type="revolute">
             <origin xyz="${front_hind*hip_j_com_x} ${mirror*hip_j_com_y} ${hip_j_com_z}" rpy="0 0 0" />
             <parent link="${name}_hip_link"/>
@@ -143,5 +143,5 @@
         </link>
         <!-- KFE_joint -->
-        <joint name="${name}_KFE_joint" type="revolute">
+        <joint name="${name}_KFE" type="revolute">
             <origin xyz="${front_hind*knee_j_com_x} ${mirror*knee_j_com_y} ${knee_j_com_z}" rpy="0 0 0" />
             <parent link="${name}_thigh_link"/>

File: legged_examples/legged_xterra/legged_xterra_description/urdf/common/transmission.xacro (robot description, xacro)
@@ -4,5 +4,5 @@
         <transmission name="${name}_HAA_tran">
             <type>transmission_interface/SimpleTransmission</type>
-            <joint name="${name}_HAA_joint">
+            <joint name="${name}_HAA">
                 <hardwareInterface>hardware_interface/EffortJointInterface</hardwareInterface>
             </joint>
@@ -14,5 +14,5 @@
         <transmission name="${name}_HFE_tran">
             <type>transmission_interface/SimpleTransmission</type>
-            <joint name="${name}_HFE_joint">
+            <joint name="${name}_HFE">
                 <hardwareInterface>hardware_interface/EffortJointInterface</hardwareInterface>
             </joint>
@@ -24,5 +24,5 @@
         <transmission name="${name}_KFE_tran">
             <type>transmission_interface/SimpleTransmission</type>
-            <joint name="${name}_KFE_joint">
+            <joint name="${name}_KFE">
                 <hardwareInterface>hardware_interface/EffortJointInterface</hardwareInterface>
             </joint>

File: legged_examples/legged_xterra/legged_xterra_description/urdf/robot.xacro (robot description, xacro)
@@ -32,7 +32,7 @@
     </link>
     <xacro:IMU connected_to="base" imu_name="base_imu" xyz="0. 0. 0." rpy="0. 0. 0."/>
-    <xacro:leg name="FR" mirror="1" front_hind="1"  />
-    <xacro:leg name="FL" mirror="-1"  front_hind="1"  />
-    <xacro:leg name="RR" mirror="1" front_hind="-1" />
-    <xacro:leg name="RL" mirror="-1"  front_hind="-1" />
+    <xacro:leg name="RF" mirror="1" front_hind="1"  />
+    <xacro:leg name="LF" mirror="-1"  front_hind="1"  />
+    <xacro:leg name="RH" mirror="1" front_hind="-1" />
+    <xacro:leg name="LH" mirror="-1"  front_hind="-1" />
 </robot>
