Commit message: Added DIDC (kinda working, still testing + checking) and modified some MPC parameters. Need more tuning and proper sanitization for sending commands before integrating this into QL

File: legged_examples/legged_unitree/legged_unitree_description/urdf/go2/const.xacro (robot description, xacro)
@@ -12,8 +12,10 @@
     <xacro:property name="thigh_shoulder_radius" value="0.041"/>
     <xacro:property name="thigh_shoulder_length" value="0.032"/>
-    <xacro:property name="thigh_shoulder_y_offset" value="-0.0"/>
+    <xacro:property name="thigh_shoulder_y_offset" value="0.0465"/>
+    <xacro:property name="thigh_shoulder_x_offset" value="0.1934"/>
     <xacro:property name="thigh_width" value="0.0245"/>
     <xacro:property name="thigh_height" value="0.034"/>
     <xacro:property name="thigh_x_offset" value="-0.0"/>
+    <xacro:property name="thigh_y_offset" value="-0.0955"/>
     <xacro:property name="calf_width" value="0.016"/>
     <xacro:property name="calf_height" value="0.016"/>

Commit message: Fixed the task.info for M2. Using wrong link inertias for now. Need to fix that.

File: legged_examples/legged_unitree/legged_unitree_description/urdf/go2/const.xacro (robot description, xacro)
@@ -68,5 +68,5 @@
     <xacro:property name="trunk_ixz" value="0.0014849"/>
     <xacro:property name="trunk_iyy" value="0.098077"/>
-    <xacro:property name="trunk_iyz" value="-3.12E-05"/>
+    <xacro:property name="trunk_iyz" value="-0.0000312"/>
     <xacro:property name="trunk_izz" value="0.107"/>
     <!-- hip (left front) -->
@@ -76,8 +76,8 @@
     <xacro:property name="hip_com_z" value="-0.000105"/>
     <xacro:property name="hip_ixx" value="0.00048"/>
-    <xacro:property name="hip_ixy" value="-3.01E-06"/>
-    <xacro:property name="hip_ixz" value="1.11E-06"/>
+    <xacro:property name="hip_ixy" value="-0.00000301"/>
+    <xacro:property name="hip_ixz" value="0.00000111"/>
     <xacro:property name="hip_iyy" value="0.000884"/>
-    <xacro:property name="hip_iyz" value="-1.42E-06"/>
+    <xacro:property name="hip_iyz" value="-0.00000142"/>
     <xacro:property name="hip_izz" value="0.000596"/>
     <!-- thigh -->
@@ -87,5 +87,5 @@
     <xacro:property name="thigh_com_z" value="-0.0327"/>
     <xacro:property name="thigh_ixx" value="0.00584"/>
-    <xacro:property name="thigh_ixy" value="8.72E-05"/>
+    <xacro:property name="thigh_ixy" value="0.0000872"/>
     <xacro:property name="thigh_ixz" value="-0.000289"/>
     <xacro:property name="thigh_iyy" value="0.0058"/>
@@ -98,9 +98,9 @@
     <xacro:property name="calf_com_z" value="-0.115"/>
     <xacro:property name="calf_ixx" value="0.00108"/>
-    <xacro:property name="calf_ixy" value="3.4E-07"/>
-    <xacro:property name="calf_ixz" value="1.72E-05"/>
+    <xacro:property name="calf_ixy" value="0.00000034"/>
+    <xacro:property name="calf_ixz" value="0.0000172"/>
     <xacro:property name="calf_iyy" value="0.0011"/>
-    <xacro:property name="calf_iyz" value="8.28E-06"/>
-    <xacro:property name="calf_izz" value="3.29E-05"/>
+    <xacro:property name="calf_iyz" value="0.00000828"/>
+    <xacro:property name="calf_izz" value="0.0000329"/>
     <!-- foot -->
     <xacro:property name="foot_mass" value="0.06"/>

File: legged_examples/legged_xterra/legged_xterra_description/urdf/m2/const.xacro (robot description, xacro)
@@ -45,5 +45,5 @@
     <!-- joint limits -->
     <xacro:property name="damping" value="0"/>
-    <xacro:property name="friction" value="0.2"/>
+    <xacro:property name="friction" value="0.0"/>
     <xacro:property name="hip_position_max" value="1.0472"/>
     <xacro:property name="hip_position_min" value="-1.0472"/>
@@ -60,47 +60,47 @@
     <!-- dynamics inertial value -->
     <!-- trunk -->
-    <xacro:property name="trunk_mass" value="5.18596663"/>
-    <xacro:property name="trunk_com_x" value="0.00918208"/>
-    <xacro:property name="trunk_com_y" value="-0.00133606"/>
-    <xacro:property name="trunk_com_z" value="-0.00430117"/>
-    <xacro:property name="trunk_ixx" value="0.02220107"/>
-    <xacro:property name="trunk_ixy" value="-0.00019966"/>
-    <xacro:property name="trunk_ixz" value="-0.00048929"/>
-    <xacro:property name="trunk_iyy" value="0.05026338"/>
-    <xacro:property name="trunk_iyz" value="-0.00001273"/>
-    <xacro:property name="trunk_izz" value="0.06413613"/>
+    <xacro:property name="trunk_mass" value="6.921"/>
+    <xacro:property name="trunk_com_x" value="0.021112"/>
+    <xacro:property name="trunk_com_y" value="0.00"/>
+    <xacro:property name="trunk_com_z" value="-0.005366"/>
+    <xacro:property name="trunk_ixx" value="0.02448"/>
+    <xacro:property name="trunk_ixy" value="0.00012166"/>
+    <xacro:property name="trunk_ixz" value="0.0014849"/>
+    <xacro:property name="trunk_iyy" value="0.098077"/>
+    <xacro:property name="trunk_iyz" value="-0.0000312"/>
+    <xacro:property name="trunk_izz" value="0.107"/>
     <!-- hip (left front) -->
-    <xacro:property name="thigh_mass" value="0.15396568"/>
-    <xacro:property name="thigh_com_x" value="0.00000000"/>
-    <xacro:property name="thigh_com_y" value="-0.00262472"/>
-    <xacro:property name="thigh_com_z" value="-0.06933846"/>
-    <xacro:property name="thigh_ixx" value="0.00075104"/>
-    <xacro:property name="thigh_ixy" value="0.00000000"/>
-    <xacro:property name="thigh_ixz" value="0.00000000"/>
-    <xacro:property name="thigh_iyy" value="0.00076325"/>
-    <xacro:property name="thigh_iyz" value="-0.00002968"/>
-    <xacro:property name="thigh_izz" value="0.00004729"/>
+    <xacro:property name="hip_mass" value="0.678"/>
+    <xacro:property name="hip_com_x" value="-0.0054"/>
+    <xacro:property name="hip_com_y" value="0.00194"/>
+    <xacro:property name="hip_com_z" value="-0.000105"/>
+    <xacro:property name="hip_ixx" value="0.00048"/>
+    <xacro:property name="hip_ixy" value="-0.00000301"/>
+    <xacro:property name="hip_ixz" value="0.00000111"/>
+    <xacro:property name="hip_iyy" value="0.000884"/>
+    <xacro:property name="hip_iyz" value="-0.00000142"/>
+    <xacro:property name="hip_izz" value="0.000596"/>
     <!-- thigh -->
-    <xacro:property name="hip_mass" value="1.12704463"/>
-    <xacro:property name="hip_com_x" value="0.04244851"/>
-    <xacro:property name="hip_com_y" value="-0.07733848"/>
-    <xacro:property name="hip_com_z" value="0.00084768"/>
-    <xacro:property name="hip_ixx" value="0.0026019"/>
-    <xacro:property name="hip_ixy" value="0.0001226"/>
-    <xacro:property name="hip_ixz" value="0.0000075"/>
-    <xacro:property name="hip_iyy" value="0.0009202"/>
-    <xacro:property name="hip_iyz" value="-0.0000024"/>
-    <xacro:property name="hip_izz" value="0.0026365"/>
+    <xacro:property name="thigh_mass" value="1.152"/>
+    <xacro:property name="thigh_com_x" value="-0.00374"/>
+    <xacro:property name="thigh_com_y" value="-0.0223"/>
+    <xacro:property name="thigh_com_z" value="-0.0327"/>
+    <xacro:property name="thigh_ixx" value="0.00584"/>
+    <xacro:property name="thigh_ixy" value="0.0000872"/>
+    <xacro:property name="thigh_ixz" value="-0.000289"/>
+    <xacro:property name="thigh_iyy" value="0.0058"/>
+    <xacro:property name="thigh_iyz" value="0.000808"/>
+    <xacro:property name="thigh_izz" value="0.00103"/>
     <!-- calf -->
-    <xacro:property name="calf_mass" value="0.1244820"/>
-    <xacro:property name="calf_com_x" value="-0.0010600"/>
-    <xacro:property name="calf_com_y" value="0.0000090"/>
-    <xacro:property name="calf_com_z" value="-0.0450013"/>
-    <xacro:property name="calf_ixx" value="0.0005021"/>
-    <xacro:property name="calf_ixy" value="0.0000000"/>
-    <xacro:property name="calf_ixz" value="-0.0000127"/>
-    <xacro:property name="calf_iyy" value="0.0005174"/>
-    <xacro:property name="calf_iyz" value="0.0000001"/>
-    <xacro:property name="calf_izz" value="0.0000202"/>
+    <xacro:property name="calf_mass" value="0.154"/>
+    <xacro:property name="calf_com_x" value="0.00548"/>
+    <xacro:property name="calf_com_y" value="-0.000975"/>
+    <xacro:property name="calf_com_z" value="-0.115"/>
+    <xacro:property name="calf_ixx" value="0.00108"/>
+    <xacro:property name="calf_ixy" value="0.00000034"/>
+    <xacro:property name="calf_ixz" value="0.0000172"/>
+    <xacro:property name="calf_iyy" value="0.0011"/>
+    <xacro:property name="calf_iyz" value="0.00000828"/>
+    <xacro:property name="calf_izz" value="0.0000329"/>
     <!-- foot -->
     <xacro:property name="foot_mass" value="0.02330447"/>
