Commit message: Updated const.xacro, still have to update thigh offset in an axis

File: legged_examples/legged_xterra/legged_xterra_description/urdf/m2/const.xacro (robot description, xacro)
@@ -7,23 +7,23 @@
     <xacro:property name="trunk_width" value="0.12"/>
     <xacro:property name="trunk_length" value="0.294"/>
-    <xacro:property name="trunk_height" value="0.114"/>
-    <xacro:property name="hip_radius" value="0.046"/>
+    <xacro:property name="trunk_height" value="0.13"/>
+    <xacro:property name="hip_radius" value="0.09"/>
     <xacro:property name="hip_length" value="0.05"/>
-    <xacro:property name="thigh_shoulder_radius" value="0.041"/>
+    <xacro:property name="thigh_shoulder_radius" value="0.03"/>
     <xacro:property name="thigh_shoulder_length" value="0.05"/>
     <xacro:property name="thigh_shoulder_y_offset" value="0.07"/>
     <xacro:property name="thigh_shoulder_x_offset" value="0.147"/>
-    <xacro:property name="thigh_width" value="0.0245"/>
-    <xacro:property name="thigh_height" value="0.034"/>
+    <xacro:property name="thigh_width" value="0.037"/>
+    <xacro:property name="thigh_height" value="0.025"/>
     <xacro:property name="thigh_x_offset" value="-0.0"/>
     <xacro:property name="thigh_y_offset" value="-0.0955"/>
-    <xacro:property name="calf_width" value="0.026"/>
-    <xacro:property name="calf_height" value="0.026"/>
+    <xacro:property name="calf_width" value="0.019"/>
+    <xacro:property name="calf_height" value="0.013"/>
     <xacro:property name="calf_x_offset" value="0.0"/>
-    <xacro:property name="foot_radius" value="0.02"/>
+    <xacro:property name="foot_radius" value="0.024"/>
     <xacro:property name="stick_radius" value="0.01"/>
     <xacro:property name="stick_length" value="0.18"/>
     <!-- kinematic value -->
-    <xacro:property name="thigh_offset" value="0.0955"/>
+    <xacro:property name="thigh_offset" value="0.081"/>
     <xacro:property name="thigh_length" value="0.19"/>
     <xacro:property name="calf_length" value="0.19"/>
@@ -34,9 +34,9 @@
     <xacro:property name="hip_offset" value="0.0955"/>
     <!-- offset of link locations (left front) incremental from base/wrt joint -->
-    <xacro:property name="hip_offset_x" value="0.147"/>
+    <xacro:property name="hip_offset_x" value="0.127"/>
     <xacro:property name="hip_offset_y" value="0.06"/>
     <xacro:property name="hip_offset_z" value="0.0"/>
-    <xacro:property name="thigh_offset_x" value="0"/>
-    <xacro:property name="thigh_offset_y" value="0.07"/>
+    <xacro:property name="thigh_offset_x" value="0.081"/>
+    <xacro:property name="thigh_offset_y" value="0.08"/>
     <xacro:property name="thigh_offset_z" value="0.0"/>
     <xacro:property name="calf_offset_x" value="0.0"/>
@@ -44,64 +44,64 @@
     <xacro:property name="calf_offset_z" value="-0.19"/>
     <!-- joint limits -->
-    <xacro:property name="damping" value="0.0"/>
-    <xacro:property name="friction" value="0.0"/>
+    <xacro:property name="damping" value="750"/>
+    <xacro:property name="friction" value="0.3"/>
     <xacro:property name="hip_position_max" value="1.0472"/>
     <xacro:property name="hip_position_min" value="-1.0472"/>
-    <xacro:property name="hip_velocity_max" value="30.1"/>
+    <xacro:property name="hip_velocity_max" value="28.6"/>
     <xacro:property name="hip_torque_max" value="23.7"/>
     <xacro:property name="thigh_position_max" value="3.4907"/>
     <xacro:property name="thigh_position_min" value="-1.5708"/>
-    <xacro:property name="thigh_velocity_max" value="30.1"/>
+    <xacro:property name="thigh_velocity_max" value="52.4"/>
     <xacro:property name="thigh_torque_max" value="23.7"/>
     <xacro:property name="calf_position_max" value="-0.83776"/>
     <xacro:property name="calf_position_min" value="-2.7227"/>
-    <xacro:property name="calf_velocity_max" value="20.06"/>
+    <xacro:property name="calf_velocity_max" value="28.6"/>
     <xacro:property name="calf_torque_max" value="35.55"/>
     <!-- dynamics inertial value -->
     <!-- trunk -->
-    <xacro:property name="trunk_mass" value="6.921"/>
-    <xacro:property name="trunk_com_x" value="0.021112"/>
-    <xacro:property name="trunk_com_y" value="0.00"/>
-    <xacro:property name="trunk_com_z" value="-0.005366"/>
-    <xacro:property name="trunk_ixx" value="0.02448"/>
-    <xacro:property name="trunk_ixy" value="0.00012166"/>
-    <xacro:property name="trunk_ixz" value="0.0014849"/>
-    <xacro:property name="trunk_iyy" value="0.098077"/>
-    <xacro:property name="trunk_iyz" value="-3.12E-05"/>
-    <xacro:property name="trunk_izz" value="0.107"/>
+    <xacro:property name="trunk_mass" value="5.18596663"/>
+    <xacro:property name="trunk_com_x" value="0.00918208"/>
+    <xacro:property name="trunk_com_y" value="-0.00133606"/>
+    <xacro:property name="trunk_com_z" value="-0.00430117"/>
+    <xacro:property name="trunk_ixx" value="0.02220107"/>
+    <xacro:property name="trunk_ixy" value="-0.00019966"/>
+    <xacro:property name="trunk_ixz" value="-0.00048929"/>
+    <xacro:property name="trunk_iyy" value="0.05026338"/>
+    <xacro:property name="trunk_iyz" value="-0.00001273"/>
+    <xacro:property name="trunk_izz" value="0.06413613"/>
     <!-- hip (left front) -->
-    <xacro:property name="hip_mass" value="0.678"/>
-    <xacro:property name="hip_com_x" value="-0.0054"/>
-    <xacro:property name="hip_com_y" value="0.00194"/>
-    <xacro:property name="hip_com_z" value="-0.000105"/>
-    <xacro:property name="hip_ixx" value="0.00048"/>
-    <xacro:property name="hip_ixy" value="-3.01E-06"/>
-    <xacro:property name="hip_ixz" value="1.11E-06"/>
-    <xacro:property name="hip_iyy" value="0.000884"/>
-    <xacro:property name="hip_iyz" value="-1.42E-06"/>
-    <xacro:property name="hip_izz" value="0.000596"/>
+    <xacro:property name="hip_mass" value="0.15396568"/>
+    <xacro:property name="hip_com_x" value="0.00000000"/>
+    <xacro:property name="hip_com_y" value="-0.00262472"/>
+    <xacro:property name="hip_com_z" value="-0.06933846"/>
+    <xacro:property name="hip_ixx" value="0.00075104"/>
+    <xacro:property name="hip_ixy" value="0.00000000"/>
+    <xacro:property name="hip_ixz" value="0.00000000"/>
+    <xacro:property name="hip_iyy" value="0.00076325"/>
+    <xacro:property name="hip_iyz" value="-0.00002968"/>
+    <xacro:property name="hip_izz" value="0.00004729"/>
     <!-- thigh -->
-    <xacro:property name="thigh_mass" value="1.152"/>
-    <xacro:property name="thigh_com_x" value="-0.00374"/>
-    <xacro:property name="thigh_com_y" value="-0.0223"/>
-    <xacro:property name="thigh_com_z" value="-0.0327"/>
-    <xacro:property name="thigh_ixx" value="0.00584"/>
-    <xacro:property name="thigh_ixy" value="8.72E-05"/>
-    <xacro:property name="thigh_ixz" value="-0.000289"/>
-    <xacro:property name="thigh_iyy" value="0.0058"/>
-    <xacro:property name="thigh_iyz" value="0.000808"/>
-    <xacro:property name="thigh_izz" value="0.00103"/>
+    <xacro:property name="thigh_mass" value="1.12704463"/>
+    <xacro:property name="thigh_com_x" value="0.04244851"/>
+    <xacro:property name="thigh_com_y" value="-0.07733848"/>
+    <xacro:property name="thigh_com_z" value="0.00084768"/>
+    <xacro:property name="thigh_ixx" value="0.0026019"/>
+    <xacro:property name="thigh_ixy" value="0.0001226"/>
+    <xacro:property name="thigh_ixz" value="0.0000075"/>
+    <xacro:property name="thigh_iyy" value="0.0009202"/>
+    <xacro:property name="thigh_iyz" value="-0.0000024"/>
+    <xacro:property name="thigh_izz" value="0.0026365"/>
     <!-- calf -->
-    <xacro:property name="calf_mass" value="0.154"/>
-    <xacro:property name="calf_com_x" value="0.00548"/>
-    <xacro:property name="calf_com_y" value="-0.000975"/>
-    <xacro:property name="calf_com_z" value="-0.115"/>
-    <xacro:property name="calf_ixx" value="0.00108"/>
-    <xacro:property name="calf_ixy" value="3.4E-07"/>
-    <xacro:property name="calf_ixz" value="1.72E-05"/>
-    <xacro:property name="calf_iyy" value="0.0011"/>
-    <xacro:property name="calf_iyz" value="8.28E-06"/>
-    <xacro:property name="calf_izz" value="3.29E-05"/>
+    <xacro:property name="calf_mass" value="0.1244820"/>
+    <xacro:property name="calf_com_x" value="-0.0010600"/>
+    <xacro:property name="calf_com_y" value="0.0000090"/>
+    <xacro:property name="calf_com_z" value="-0.0450013"/>
+    <xacro:property name="calf_ixx" value="0.0005021"/>
+    <xacro:property name="calf_ixy" value="0.0000000"/>
+    <xacro:property name="calf_ixz" value="-0.0000127"/>
+    <xacro:property name="calf_iyy" value="0.0005174"/>
+    <xacro:property name="calf_iyz" value="0.0000001"/>
+    <xacro:property name="calf_izz" value="0.0000202"/>
     <!-- foot -->
-    <xacro:property name="foot_mass" value="0.06"/>
+    <xacro:property name="foot_mass" value="0.02330447"/>
 </robot>

Commit message: fixed hip and trunk masses and com

File: legged_examples/legged_xterra/legged_xterra_description/urdf/m2/const.xacro (robot description, xacro)
@@ -60,8 +60,8 @@
     <!-- dynamics inertial value -->
     <!-- trunk -->
-    <xacro:property name="trunk_mass" value="6.921"/>
-    <xacro:property name="trunk_com_x" value="0.021112"/>
-    <xacro:property name="trunk_com_y" value="0.00"/>
-    <xacro:property name="trunk_com_z" value="-0.005366"/>
+    <xacro:property name="trunk_mass" value="5.18596663"/>
+    <xacro:property name="trunk_com_x" value="0.00918208"/>
+    <xacro:property name="trunk_com_y" value="-0.00133606"/>
+    <xacro:property name="trunk_com_z" value="-0.00430117"/>
     <xacro:property name="trunk_ixx" value="0.02448"/>
     <xacro:property name="trunk_ixy" value="0.00012166"/>
@@ -71,8 +71,8 @@
     <xacro:property name="trunk_izz" value="0.107"/>
     <!-- hip (left front) -->
-    <xacro:property name="hip_mass" value="0.678"/>
-    <xacro:property name="hip_com_x" value="-0.0054"/>
-    <xacro:property name="hip_com_y" value="0.00194"/>
-    <xacro:property name="hip_com_z" value="-0.000105"/>
+    <xacro:property name="hip_mass" value="1.12704463"/>
+    <xacro:property name="hip_com_x" value="0.04244851"/>
+    <xacro:property name="hip_com_y" value="-0.07733848"/>
+    <xacro:property name="hip_com_z" value="0.00084768"/>
     <xacro:property name="hip_ixx" value="0.00048"/>
     <xacro:property name="hip_ixy" value="-0.00000301"/>

Commit message: Fixed mass, com & inertia values for links, except calf;

File: legged_examples/legged_xterra/legged_xterra_description/urdf/m2/const.xacro (robot description, xacro)
@@ -64,10 +64,10 @@
     <xacro:property name="trunk_com_y" value="-0.00133606"/>
     <xacro:property name="trunk_com_z" value="-0.00430117"/>
-    <xacro:property name="trunk_ixx" value="0.02448"/>
-    <xacro:property name="trunk_ixy" value="0.00012166"/>
-    <xacro:property name="trunk_ixz" value="0.0014849"/>
-    <xacro:property name="trunk_iyy" value="0.098077"/>
-    <xacro:property name="trunk_iyz" value="-0.0000312"/>
-    <xacro:property name="trunk_izz" value="0.107"/>
+    <xacro:property name="trunk_ixx" value="0.02220107"/>
+    <xacro:property name="trunk_ixy" value="-0.00019966"/>
+    <xacro:property name="trunk_ixz" value="-0.00048929"/>
+    <xacro:property name="trunk_iyy" value="0.05026338"/>
+    <xacro:property name="trunk_iyz" value="-0.00001273"/>
+    <xacro:property name="trunk_izz" value="0.06413613"/>
     <!-- hip (left front) -->
     <xacro:property name="hip_mass" value="1.12704463"/>
@@ -75,25 +75,25 @@
     <xacro:property name="hip_com_y" value="-0.07733848"/>
     <xacro:property name="hip_com_z" value="0.00084768"/>
-    <xacro:property name="hip_ixx" value="0.00048"/>
-    <xacro:property name="hip_ixy" value="-0.00000301"/>
-    <xacro:property name="hip_ixz" value="0.00000111"/>
-    <xacro:property name="hip_iyy" value="0.000884"/>
-    <xacro:property name="hip_iyz" value="-0.00000142"/>
-    <xacro:property name="hip_izz" value="0.000596"/>
+    <xacro:property name="hip_ixx" value="0.0026019"/>
+    <xacro:property name="hip_ixy" value="0.0001226"/>
+    <xacro:property name="hip_ixz" value="0.0000075"/>
+    <xacro:property name="hip_iyy" value="0.0009202"/>
+    <xacro:property name="hip_iyz" value="-0.0000024"/>
+    <xacro:property name="hip_izz" value="0.0026365"/>
     <!-- thigh -->
-    <xacro:property name="thigh_mass" value="1.152"/>
-    <xacro:property name="thigh_com_x" value="-0.00374"/>
-    <xacro:property name="thigh_com_y" value="-0.0223"/>
-    <xacro:property name="thigh_com_z" value="-0.0327"/>
-    <xacro:property name="thigh_ixx" value="0.00584"/>
-    <xacro:property name="thigh_ixy" value="0.0000872"/>
-    <xacro:property name="thigh_ixz" value="-0.000289"/>
-    <xacro:property name="thigh_iyy" value="0.0058"/>
-    <xacro:property name="thigh_iyz" value="0.000808"/>
-    <xacro:property name="thigh_izz" value="0.00103"/>
+    <xacro:property name="thigh_mass" value="0.15396568"/>
+    <xacro:property name="thigh_com_x" value="0.0"/>
+    <xacro:property name="thigh_com_y" value="-0.00262472"/>
+    <xacro:property name="thigh_com_z" value="-0.06933846"/>
+    <xacro:property name="thigh_ixx" value="0.00075104"/>
+    <xacro:property name="thigh_ixy" value="0.00000000"/>
+    <xacro:property name="thigh_ixz" value="0.00000000"/>
+    <xacro:property name="thigh_iyy" value="0.00076325"/>
+    <xacro:property name="thigh_iyz" value="-0.00002968"/>
+    <xacro:property name="thigh_izz" value="0.00004729"/>
     <!-- calf -->
-    <xacro:property name="calf_mass" value="0.154"/>
-    <xacro:property name="calf_com_x" value="0.00548"/>
-    <xacro:property name="calf_com_y" value="-0.000975"/>
+    <xacro:property name="calf_mass" value="0.1244820"/>
+    <xacro:property name="calf_com_x" value="-0.0010600"/>
+    <xacro:property name="calf_com_y" value="0.0000090"/>
     <xacro:property name="calf_com_z" value="-0.115"/>
     <xacro:property name="calf_ixx" value="0.00108"/>

Commit message: Added joint command and sensor data dds topics and msgs

File: legged_examples/legged_xterra/legged_xterra_description/urdf/m2/const.xacro (robot description, xacro)
@@ -97,6 +97,6 @@
     <xacro:property name="calf_com_y" value="0.0000090"/>
     <xacro:property name="calf_com_z" value="-0.115"/>
-    <xacro:property name="calf_ixx" value="0.00108"/>
-    <xacro:property name="calf_ixy" value="0.00000034"/>
+    <xacro:property name="calf_ixx" value="0.0005021"/>
+    <xacro:property name="calf_ixy" value="0.00"/>
     <xacro:property name="calf_ixz" value="0.0000172"/>
     <xacro:property name="calf_iyy" value="0.0011"/>
